File: CP 400 Color 2.kicad_pcb (KiCad board)
At the start: 2 copper layers, 255 x 170 mm, 28 parts, among them J1 Conn_02x20_Odd_Even, J2 DB9_Female, J3 DB9_Female, J4 DB9_Female, J5 DB15_Female_HighDensity_Mount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, J6 Conn_Coaxial, J7 Conn_Coaxial_Power, J8 Conn_02x22_Odd_Even, U1 MC6883, U10 EPM3064ALC44-10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

Commit message: no significant changes
Parts:
- J4: footprint Connector_BarrelJack:BarrelJack_CUI_PJ-063AH_Horizontal -> Connector_Dsub:DSUB-9_Female_Horizontal_P2.77x2.54mm_EdgePinOffset9.40mm
- J6: footprint Connector_Coaxial:BNC_Win_364A2x95_Horizontal -> Connector_BarrelJack:BarrelJack_CUI_PJ-063AH_Horizontal
- J7: value Conn_Coaxial_Power -> Conn_Coaxial; footprint Connector_BarrelJack:BarrelJack_CUI_PJ-102AH_Horizontal -> Connector_BarrelJack:BarrelJack_CUI_PJ-063AH_Horizontal
- J8: footprint Connector_PinHeader_2.54mm:PinHeader_2x22_P2.54mm_Vertical -> Connector_IDC:IDC-Header_2x20_P2.54mm_Vertical
- moved J6 13.6 mm to (262.3, 63.3), turned to 180 degrees
- moved J7 2.77 mm to (74.3, 63.5)
