File: CP 400 Color 2.kicad_sch (KiCad schematic)
At the start: 27 parts, among them J1 Conn_02x20_Odd_Even, J2 DB9_Female, J3 DB9_Female, J4 DB9_Female, J5 DB15_Female_HighDensity_Mount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, J6 Conn_Coaxial, J7 Conn_Coaxial_Power, J8 Conn_02x22_Odd_Even, U1 MC6883, U10 EPM3064ALC44-10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

Commit message: no significant changes
Parts:
- removed J7: Conn_Coaxial_Power, Connector_BarrelJack:BarrelJack_CUI_PJ-102AH_Horizontal, symbol Connector:Conn_Coaxial_Power
- added J7: Conn_Coaxial, Connector_BarrelJack:BarrelJack_CUI_PJ-063AH_Horizontal, symbol Connector:Conn_Coaxial
- J4: footprint Connector_BarrelJack:BarrelJack_CUI_PJ-063AH_Horizontal -> Connector_Dsub:DSUB-9_Female_Horizontal_P2.77x2.54mm_EdgePinOffset9.40mm
- J6: footprint Connector_Coaxial:BNC_Win_364A2x95_Horizontal -> Connector_BarrelJack:BarrelJack_CUI_PJ-063AH_Horizontal
- J8: footprint Connector_PinHeader_2.54mm:PinHeader_2x22_P2.54mm_Vertical -> Connector_IDC:IDC-Header_2x20_P2.54mm_Vertical
Changed lines of the file:
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@@
     )
-  )
-  (symbol (lib_id "Connector:Conn_Coaxial_Power") (at 207.264 246.888 0) (unit 1)
-    (in_bom yes) (on_board yes) (fields_autoplaced)
-    (property "Reference" "J7" (id 0) (at 209.55 247.1419 0)
-      (effects (font (size 1.27 1.27)) (justify left))
-    )
-    (property "Value" "Conn_Coaxial_Power" (id 1) (at 209.55 249.6819 0)
-      (effects (font (size 1.27 1.27)) (justify left))
-    )
-    (property "Footprint" "Connector_BarrelJack:BarrelJack_CUI_PJ-102AH_Horizontal" (id 2) (at 207.264 248.158 0)
-      (effects (font (size 1.27 1.27)) hide)
-    )
-    (property "Datasheet" "~" (id 3) (at 207.264 248.158 0)
-      (effects (font (size 1.27 1.27)) hide)
-    )
-    (pin "1")
-    (pin "2")
   )
   (symbol (lib_id "Interface:6821") (at 214.63 76.2 0) (unit 1)
@@
     (property "Reference" "J8" (id 0) (at 272.288 127 0))
     (property "Value" "Conn_02x22_Odd_Even" (id 1) (at 272.288 129.54 0))
-    (property "Footprint" "Connector_PinHeader_2.54mm:PinHeader_2x22_P2.54mm_Vertical" (id 2) (at 271.018 158.496 0)
+    (property "Footprint" "Connector_IDC:IDC-Header_2x20_P2.54mm_Vertical" (id 2) (at 271.018 158.496 0)
       (effects (font (size 1.27 1.27)) hide)
     )
@@
       (effects (font (size 1.27 1.27)) (justify left))
     )
-    (property "Footprint" "Connector_BarrelJack:BarrelJack_CUI_PJ-063AH_Horizontal" (id 2) (at 111.252 247.904 0)
+    (property "Footprint" "Connector_Dsub:DSUB-9_Female_Horizontal_P2.77x2.54mm_EdgePinOffset9.40mm" (id 2) (at 111.252 247.904 0)
       (effects (font (size 1.27 1.27)) hide)
     )
@@
       (effects (font (size 1.27 1.27)) (justify left))
     )
-    (property "Footprint" "Connector_Coaxial:BNC_Win_364A2x95_Horizontal" (id 2) (at 177.292 245.872 0)
+    (property "Footprint" "Connector_BarrelJack:BarrelJack_CUI_PJ-063AH_Horizontal" (id 2) (at 177.292 245.872 0)
       (effects (font (size 1.27 1.27)) hide)
     )
@@
     (pin "9")
   )
+  (symbol (lib_id "Connector:Conn_Coaxial") (at 204.47 246.126 0) (unit 1)
+    (in_bom yes) (on_board yes) (fields_autoplaced)
+    (property "Reference" "J7" (id 0) (at 207.01 245.1491 0)
+      (effects (font (size 1.27 1.27)) (justify left))
+    )
+    (property "Value" "Conn_Coaxial" (id 1) (at 207.01 247.6891 0)
+      (effects (font (size 1.27 1.27)) (justify left))
+    )
+    (property "Footprint" "Connector_BarrelJack:BarrelJack_CUI_PJ-063AH_Horizontal" (id 2) (at 204.47 246.126 0)
+      (effects (font (size 1.27 1.27)) hide)
+    )
+    (property "Datasheet" " ~" (id 3) (at 204.47 246.126 0)
+      (effects (font (size 1.27 1.27)) hide)
+    )
+    (pin "1")
+    (pin "2")
+  )
   (sheet_instances
     (path "/" (page "1"))
@@
     )
     (path "/67a30add-0127-41b3-af24-fb67b7fe19b6"
-      (reference "J4") (unit 1) (value "DB9_Female") (footprint "Connector_BarrelJack:BarrelJack_CUI_PJ-063AH_Horizontal")
+      (reference "J4") (unit 1) (value "DB9_Female") (footprint "Connector_Dsub:DSUB-9_Female_Horizontal_P2.77x2.54mm_EdgePinOffset9.40mm")
     )
     (path "/2e8037c5-8231-4691-9ee1-e22e281c7a3c"
@@
     )
     (path "/c003701f-8655-47f1-9147-dd278b238b9c"
-      (reference "J6") (unit 1) (value "Conn_Coaxial") (footprint "Connector_Coaxial:BNC_Win_364A2x95_Horizontal")
-    )
-    (path "/3ecc83f9-f2c0-465d-85eb-235ada0406ab"
-      (reference "J7") (unit 1) (value "Conn_Coaxial_Power") (footprint "Connector_BarrelJack:BarrelJack_CUI_PJ-102AH_Horizontal")
+      (reference "J6") (unit 1) (value "Conn_Coaxial") (footprint "Connector_BarrelJack:BarrelJack_CUI_PJ-063AH_Horizontal")
+    )
+    (path "/fb23f4fd-b33d-4646-8dd5-ab698b5cf01e"
+      (reference "J7") (unit 1) (value "Conn_Coaxial") (footprint "Connector_BarrelJack:BarrelJack_CUI_PJ-063AH_Horizontal")
     )
     (path "/4d97ca6e-be0b-498f-887e-d06a23e0cf02"
-      (reference "J8") (unit 1) (value "Conn_02x22_Odd_Even") (footprint "Connector_PinHeader_2.54mm:PinHeader_2x22_P2.54mm_Vertical")
+      (reference "J8") (unit 1) (value "Conn_02x22_Odd_Even") (footprint "Connector_IDC:IDC-Header_2x20_P2.54mm_Vertical")
     )
     (path "/5f82ccb4-d94e-4303-b427-9b3cec0cf2f2"
