File: CP 400 COLOR.kicad_sch (KiCad schematic)
At the start: 228 parts, among them CN10 CN10, CN13 CN13, CN2 CANAL, CN7 CP400_CN7, K1 CoCo_K1_Ferrite, P2 DIN-4, P3 RIGHT JOYSTICK, P4 LEFT JOYSTICK, P5 DIN-5_180degree, Q1 MPS3904, Q4 2N2222, U1 MC6809E, U10 MC6883, U11 74LS138, U12 MC1372P, U14 LM339, U15 LM741, U16 74LS02, U2 MC14050B, U28 ROM EXPANSION, U29 74LS02, U3 MCM68A364, U4 6821, U5 UM1285-8, U6 74LS273, U7 MC6847, U8 6821, U9 MC14529, x1 14.31818

Commit message: Added symbol 74ls183.
Parts:
- removed CI-28: 74LS138, Package_DIP:DIP-20_W7.62mm, symbol 74xx:74LS138
- added C39: C39, symbol Device:C_Small
- added C40: C40, symbol Device:C_Small
- added C44: C44, symbol Device:C_Small
- added C45: C45, symbol Device:C_Small
- added CCV-1: CV-1, symbol Device:C_Variable
- added CI-28: 74LS138, symbol Roni:CP400_74LS138
- added D15: D15, Diode_SMD:D_SOD-123, symbol Diode:1N4148W
- added D16: D16, Diode_SMD:D_SOD-123, symbol Diode:1N4148W
- added D17: D17, Diode_SMD:D_SOD-123, symbol Diode:1N4148W
- added D20: D20, Diode_SMD:D_SOD-123, symbol Diode:1N4148W
- added D21: D21, Diode_SMD:D_SOD-123, symbol Diode:1N4148W
- added R34, R?: R34, symbol Device:R_Small
- added R35: R35, symbol Device:R_Small
- added R36: R36, symbol Device:R_Small
- added R62: R62, symbol Device:R_Small
- added R?: R59, symbol Device:R_Small
- added XTAL: XTAL 1, symbol Device:Crystal
Connections:
- net +5V: now also D16.1 (K), R35.2, R36.2, R62.2, R?.2, R?.2
- net 32: now also CI-28.12 (Y3)
- net 40: now also CI-28.6 (G1), R62.1
- net E: now also D20.1 (K)
- net GNDREF: now also C39.2, C40.2, C44.2, C45.2, CCV-1.2, CI-28.5 (G2B), CI-28.8 (GND)
- net RESET: now also C44.1, D17.2 (A), R36.1
- net VCLK: now also CI-29.7 (VClk), D15.2 (A)
- net at CI-12.22 (~{OE}): now also CI-28.14 (Y1)
- net at CI-17.23 (~{CS2}): now also CI-28.10 (Y5)
- net at CI-14.23 (~{CS2}): now also CI-28.11 (Y4)
- net at CI-11.22 (~{OE}): now also CI-28.13 (Y2)
- net at CI-21.1 (~{R}): now also CI-21.2 (D), CI-21.3 (C)
- net at CI-21.4 (~{S}): now also CI-22.3, R?.1
- net at CI-21.5 (Q): now also CI-28.4 (G2A)
- net at CI-(3/4/5/6/7/8/9/10).4 (/RAS): now also CI-29.12 (/RAS)
- net at CI-29.25 (S2): now also CI-22.1, CI-28.3 (C)
- net at CI-29.26 (S1): now also CI-28.2 (B)
- net at CI-29.27 (S0): now also CI-28.1 (A)
- net at CI-29.5 (OscIn): now also C39.1, XTAL.1
- net at CI-29.6 (OscOut): now also R34.1
- net at CI-22.2: now also D20.2 (A), D21.2 (A), R?.1
- new net: C45.1, D15.1 (K), D16.2 (A), D17.1 (K), R35.1
- new net: C40.1, R34.2, XTAL.2
Other:
- note added: "C44: Electrolitico ?"
- note added: "D21: Conecta onde?"
- moved on the sheet: CI-11, CI-12, CI-14, CI-15, CI-17, CI-18, CI-21A, CI-22A

Commit message: more updates
Parts:
- added R25: R25, symbol Device:R_Small
Connections:
- net E is gone; now on net 6: CI-14.25 (ENABLE), CI-17.25 (ENABLE), D20.1 (K), U4.25 (ENABLE), U8.25 (ENABLE)
- net +5V: now also R25.2
- net 18: now also CI-29.15 (R/W)
- net 19: now also CI-29.16 (A0)
- net 20: now also CI-29.17 (A1)
- net 21: now also CI-29.18 (A2)
- net 22: now also CI-29.19 (A3)
- net 23: now also CI-29.21 (A4)
- net 24: now also CI-29.22 (A5)
- net 25: now also CI-29.23 (A6)
- net 26: now also CI-29.24 (A7)
- net 27: now also CI-29.4 (A8)
- net 28: now also CI-29.3 (A9)
- net 29: now also CI-29.2 (A10)
- net 30: now also CI-29.1 (A11)
- net 31: now also CI-29.39 (A12)
- net 37: now also CI-29.38 (A13)
- net 38: now also CI-29.37 (A14)
- net 39: now also CI-29.36 (A15)
- net 5: now also CI-15.37 (~{RESET})
- net 6: now also CI-29.14 (E)
- net 7: now also CI-29.13 (Q)
- net DA0: now also CI-24.22 (DA0), CI-29.8 (DA0)
- net HI: now also R25.1
- net RESET: no longer CI-15.37 (~{RESET})
- net /HS: now also CI-21.11 (C), CI-24.38 (/HS), CI-27.2 (B), CI-29.9 (/HS)
- net /CAS: now reaches CI-(3/4/5/6/7/8/9/10).15 (/CAS), CI-29.11 (/CAS)
- net /WE: now reaches CI-(3/4/5/6/7/8/9/10).3 (/WR), CI-29.10 (/WE)
- net at CI-(3/4/5/6/7/8/9/10).4 (/RAS): now also CI-29.12 (/RAS)
Other:
- moved on the sheet: CI-15

Commit message: Added CP400_14529 and Joystick schema
Parts:
- removed CI-18: 4050, symbol Roni:CP400_4050B
- added C2: C2, symbol Device:C_Small
- added C3: C3, symbol Device:C_Small
- added C33: C33, symbol Device:C_Small
- added C34: C34, symbol Device:C_Small
- added C4: C4, symbol Device:C_Small
- added C5: C5, symbol Device:C_Small
- added C6: C6, symbol Device:C_Small
- added CI-15: 14529, symbol Roni:CP400_14529
- added CI-18: 14050B, symbol Roni:CP400_14050B
- added CN5: JOYESQ, symbol Connector:DIN-5
- added CN6: JOYDIR, symbol Connector:DIN-5
- added CN?: CN12, symbol Connector:Conn_01x03_Male
- added R26: R26, symbol Device:R_Small
- added R29: R29, symbol Device:R_Small
- added R30: R30, symbol Device:R_Small
- added R4: R4, symbol Device:R_Small
- added TR?: TR1, Package_TO_SOT_THT:TO-92, symbol Transistor_BJT:MPSA42
- added U?: CP400_14050B, symbol Roni:CP400_14050B
- C42: renamed from C?; value C6 -> C42
Connections:
- net +5V: now also R22.2, CI-15.16 (VDD), CI-18.1, CN?.3 (Pin_3), R4.1
- net GNDREF: now also C2.2, C3.2, C33.2, C34.2, C4.2, C5.2, C6.2, CI-15.8 (VSS), CI-18.8, CN5.3, CN6.3, TR?.1 (E)
- net HI: now also CI-15.1 (STX), CN?.1 (Pin_1)
- net at R44.1: now also CI-18.2
- net at R22.1, R44.2: now also C42.1, R41.2, R42.2, R43.2, R46.2, R54.2
- net at CI-17.10 (PB0): now also CI-17.11 (PB1), R29.1
- net at CI-17.12 (PB2): now also CN?.2 (Pin_2)
- net at CI-17.19 (CB2): now also CI-15.15 (STY)
- net at CI-17.39 (CA2): now also R26.1
- net at CI-17.4 (PA2): now also CI-18.14
- net at CI-17.5 (PA3): now also CI-18.11
- net at CI-17.6 (PA4): now also CI-18.9
- net at CI-17.7 (PA5): now also CI-18.7
- net at CI-17.8 (PA6): now also CI-18.5
- net at CI-17.9 (PA7): now also CI-18.3
- net at R42.1: now also CI-18.10
- net at R46.1: now also CI-18.12
- net at R54.1: now also CI-18.6
- net at R41.1: now also CI-18.4
- net at CI-(3/4/5/6/7/8/9/10).4 (/RAS): now also CI-29.12 (/RAS)
- net at R43.1: now also CI-18.15
- new net: R26.2, TR?.2 (B)
- new net: C4.1, CI-15.2 (X0), CN6.5
- new net: C5.1, CI-15.3 (X1), CN6.4
- new net: C6.1, CN5.1, CN6.1, R4.2
- new net: CI-15.10 (W), R29.2, R30.1
- new net: C2.1, CI-15.5 (X3), CN5.4
- new net: C3.1, CI-15.4 (X2), CN5.5
- new net L2 & FOGOD: C33.1, CN6.2
- new net L3 & FOGOE: C34.1, CN5.2
Other:
- note added: "CN12 Ligado a +5V ?"

Commit message: Continuing drawing schematic
Parts:
- added C15: C16, symbol Device:C_Small
- added CI-16, U?: LM339, symbol Comparator:LM339
- added CI-20, CI-?: LM741, symbol Amplifier_Operational:LM741
- added CN4: RS232, symbol Connector:DIN-4
- added D16: D16, Diode_SMD:D_SOD-123, symbol Diode:1N4148W
- added D19: D19, Diode_SMD:D_SOD-123, symbol Diode:1N4148W
- added R27: R27, symbol Device:R_Small
- added R32: R32, symbol Device:R_Small
- added R33: R33, symbol Device:R_Small
- added R56: R56, symbol Device:R_Small
- added R57, R?: R57, symbol Device:R_Small
- added R6: R6, symbol Device:R_Small
- added R63: R63, symbol Device:R_Small
- added R64: R64, symbol Device:R_Small
- added R65: R65, symbol Device:R_Small
- added R66: R66, symbol Device:R_Small
- added R67: R67, symbol Device:R_Small
- added R68: R68, symbol Device:R_Small
- added R69: R69, symbol Device:R_Small
- added R70: R70, symbol Device:R_Small
- added R71: R71, symbol Device:R_Small
- added R72: R72, symbol Device:R_Small
- added R75: R75, symbol Device:R_Small
Connections:
- net +12V: now also CI-20.7 (V+)
- net +5V: now also R32.2, R56.2, R65.2, R67.2, R70.2, R71.1
- net -12V: now also CI-20.4 (V-)
- net GNDREF: now also CI-15.11 (Y3), CN4.2, R33.1, R63.1, R64.1, R68.1, R69.1; no longer C33.2, C34.2, CI-15.8 (VSS)
- net HI: no longer CI-15.1 (STX)
- net at C4.1, CN6.5: no longer CI-15.2 (X0)
- net at CI-17.11 (PB1), R29.1: no longer CI-17.10 (PB0)
- net at CI-17.3 (PA1): now also CI-20.2 (-), R33.2
- net at C5.1, CN6.4: no longer CI-15.3 (X1)
- net at C2.1, CN5.4: no longer CI-15.5 (X3)
- net at CI-1.10 (CHI): now also R6.2
- net at CI-1.8 (CMO): now also C15.2
- net at C3.1, CN5.5: no longer CI-15.4 (X2)
- net at CI-15.14 (Y0): now also CI-16.8 (-)
- net at CI-15.9 (Z): now also R75.1
- net at CI-(3/4/5/6/7/8/9/10).4 (/RAS): now also CI-29.12 (/RAS)
- new net: CI-16.5 (+), R57.1, R69.2, R70.1
- new net: CI-16.2, R56.1, R57.2
- new net: CI-16.4 (-), D16.1 (K), R63.2
- new net: CI-16.1, CI-17.10 (PB0), R65.1, R66.2
- new net: CN4.1, R27.2
- new net: CN4.3, D19.2 (A)
- new net: CN4.4, D16.2 (A)
- new net: CI-16.7 (+), R66.1, R67.1, R68.2
- new net: C15.1, R6.1
- new net: CI-16.9 (+), R72.1, R75.2
- new net: CI-20.3 (+), R32.1
- new net: CI-20.6, R27.1
- new net: CI-16.14, R71.2, R72.2
- new net: CI-16.6 (-), D19.1 (K), R64.2
- no-connect marks 35 -> 37
Other:
- moved on the sheet: CI-15, CN5, CN6

Commit message: Reviewing but still incomplete schematic
Parts:
- removed C1: 1uf, Capacitor_THT:CP_Radial_D5.0mm_P2.50mm, symbol Device:C
- removed C12: 100, Capacitor_THT:CP_Radial_D5.0mm_P2.50mm, symbol Device:C
- removed C2: 10uf, Capacitor_THT:CP_Radial_D5.0mm_P2.50mm, symbol Device:C
- removed C24, C25, C41, C43: 0.1, Capacitor_THT:CP_Radial_D5.0mm_P2.50mm, symbol Device:C
- removed C3, C5: 100uf, Capacitor_THT:CP_Radial_D5.0mm_P2.50mm, symbol Device:C
- removed C4: 9.35pf, Capacitor_THT:C_Disc_D3.0mm_W2.0mm_P2.50mm, symbol Device:C_Variable
- removed C40: 0.1uf, Capacitor_THT:CP_Radial_D5.0mm_P2.50mm, symbol Device:C
- removed C42, C57, C58: 0.01, Capacitor_THT:C_Disc_D3.0mm_W2.0mm_P2.50mm, symbol Device:C
- removed C52: 20pF, Capacitor_THT:C_Disc_D3.0mm_W2.0mm_P2.50mm, symbol Device:C
- removed C53, C75: 56pF, Capacitor_THT:C_Disc_D3.0mm_W2.0mm_P2.50mm, symbol Device:C
- removed C54, C55, C56, C78, C79: 0.02, Capacitor_THT:C_Disc_D3.0mm_W2.0mm_P2.50mm, symbol Device:C
- removed C6: 25, Capacitor_THT:C_Disc_D3.0mm_W2.0mm_P2.50mm, symbol Device:C
- removed C61: 39pF, Capacitor_THT:C_Disc_D3.0mm_W2.0mm_P2.50mm, symbol Device:C
- removed C73: 56Pf, Capacitor_THT:C_Disc_D3.0mm_W2.0mm_P2.50mm, symbol Device:C
- removed C80, C81: .02uf, Capacitor_THT:C_Disc_D3.0mm_W2.0mm_P2.50mm, symbol Device:C
- removed C82: .002uf, Capacitor_THT:C_Disc_D3.0mm_W2.0mm_P2.50mm, symbol Device:C
- removed C85: 220pF, Capacitor_THT:C_Disc_D3.0mm_W2.0mm_P2.50mm, symbol Device:C
- removed CI-?: LM741, symbol Amplifier_Operational:LM741
- removed CR1, CR2, CR3, CR4, CR5, CR6, CR7: 1N4148, Diode_THT:D_DO-35_SOD27_P7.62mm_Horizontal, symbol Diode:1N4148
- removed CR10, CR9: IN982, Package_TO_SOT_THT:TO-92, symbol Device:D_Zener
- removed CR16: D_Zener, symbol Device:D_Zener
- removed CR8: 1N4002, Diode_THT:D_DO-41_SOD81_P10.16mm_Horizontal, symbol Diode:1N4002
- removed JP1, JP2, JP_RAM_SELECT1: Jumper_3_Open, symbol Jumper:Jumper_3_Open
- removed JP3: Jumper_2_Open, symbol Jumper:Jumper_2_Open
- removed K1: CoCo_K1_Ferrite, symbol Roni:CoCo_K1_Ferrite
- removed P2: DIN-4, symbol Connector:DIN-4
- removed P3: RIGHT JOYSTICK, symbol Connector:DIN-5
- removed P4: LEFT JOYSTICK, symbol Connector:DIN-5
- removed P5: DIN-5_180degree, symbol Connector:DIN-5_180degree
- removed Q1: MPS3904, Package_TO_SOT_THT:TO-92, symbol Transistor_BJT:MPSA42
- removed Q4: 2N2222, Package_TO_SOT_THT:TO-92, symbol Transistor_BJT:2N2219
- removed R1, R2, R72: 100K, Resistor_THT:R_Axial_DIN0207_L6.3mm_D2.5mm_P7.62mm_Horizontal, symbol Device:R_Small_US
- removed R10, R22, R28, R29, R48, R51, R52, R68: 10K, Resistor_THT:R_Axial_DIN0207_L6.3mm_D2.5mm_P7.62mm_Horizontal, symbol Device:R_Small_US
- removed R11: 20K, Resistor_THT:R_Axial_DIN0207_L6.3mm_D2.5mm_P7.62mm_Horizontal, symbol Device:R_Small_US
- removed R12: 40K, Resistor_THT:R_Axial_DIN0207_L6.3mm_D2.5mm_P7.62mm_Horizontal, symbol Device:R_Small_US
- removed R13: 80K, Resistor_THT:R_Axial_DIN0207_L6.3mm_D2.5mm_P7.62mm_Horizontal, symbol Device:R_Small_US
- removed R14: 162K, Resistor_THT:R_Axial_DIN0207_L6.3mm_D2.5mm_P7.62mm_Horizontal, symbol Device:R_Small_US
- removed R15: 324K, Resistor_THT:R_Axial_DIN0207_L6.3mm_D2.5mm_P7.62mm_Horizontal, symbol Device:R_Small_US
- removed R16, R23a1: 3.9K, Resistor_THT:R_Axial_DIN0207_L6.3mm_D2.5mm_P7.62mm_Horizontal, symbol Device:R_Small_US
- removed R17, R46, R73, R74, R80: 470, Resistor_THT:R_Axial_DIN0207_L6.3mm_D2.5mm_P7.62mm_Horizontal, symbol Device:R_Small_US
- removed R18: 750, Resistor_THT:R_Axial_DIN0207_L6.3mm_D2.5mm_P7.62mm_Horizontal, symbol Device:R_Small_US
- removed R19: 12K, Resistor_THT:R_Axial_DIN0207_L6.3mm_D2.5mm_P7.62mm_Horizontal, symbol Device:R_Small_US
- removed R20: 360, Resistor_THT:R_Axial_DIN0207_L6.3mm_D2.5mm_P7.62mm_Horizontal, symbol Device:R_Small_US
- removed R21: 500, Resistor_THT:R_Axial_DIN0207_L6.3mm_D2.5mm_P7.62mm_Horizontal, symbol Device:R_Potentiometer_US
- removed R23, R71: 220, Resistor_THT:R_Axial_DIN0207_L6.3mm_D2.5mm_P7.62mm_Horizontal, symbol Device:R_Small_US
- removed R24, R43, R47: 1.5K, Resistor_THT:R_Axial_DIN0207_L6.3mm_D2.5mm_P7.62mm_Horizontal, symbol Device:R_Small_US
- removed R25, R26, R30, R40, R57: 1K, Resistor_THT:R_Axial_DIN0207_L6.3mm_D2.5mm_P7.62mm_Horizontal, symbol Device:R_Small_US
- removed R27: 100 1/2W, Resistor_THT:R_Axial_DIN0207_L6.3mm_D2.5mm_P7.62mm_Horizontal, symbol Device:R_Small_US
- removed R3, R31, R32, R4, R44, R5, R6, R7: 4.7K, Resistor_THT:R_Axial_DIN0207_L6.3mm_D2.5mm_P7.62mm_Horizontal, symbol Device:R_Small_US
- removed R34: 6.2K, Resistor_THT:R_Axial_DIN0207_L6.3mm_D2.5mm_P7.62mm_Horizontal, symbol Device:R_Small_US
- removed R35: 6.8K, Resistor_THT:R_Axial_DIN0207_L6.3mm_D2.5mm_P7.62mm_Horizontal, symbol Device:R_Small_US
- removed R36, R37: 56K, Resistor_THT:R_Axial_DIN0207_L6.3mm_D2.5mm_P7.62mm_Horizontal, symbol Device:R_Small_US
- removed R38, R53, R54: 15K, Resistor_THT:R_Axial_DIN0207_L6.3mm_D2.5mm_P7.62mm_Horizontal, symbol Device:R_Small_US
- removed R39: 1.5MEG, Resistor_THT:R_Axial_DIN0207_L6.3mm_D2.5mm_P7.62mm_Horizontal, symbol Device:R_Small_US
- removed R41: 24K, Resistor_THT:R_Axial_DIN0207_L6.3mm_D2.5mm_P7.62mm_Horizontal, symbol Device:R_Small_US
- removed R42: 75K, Resistor_THT:R_Axial_DIN0207_L6.3mm_D2.5mm_P7.62mm_Horizontal, symbol Device:R_Small_US
- removed R45: 180, Resistor_THT:R_Axial_DIN0207_L6.3mm_D2.5mm_P7.62mm_Horizontal, symbol Device:R_Small_US
- removed R49, R55, R56: 10M, Resistor_THT:R_Axial_DIN0207_L6.3mm_D2.5mm_P7.62mm_Horizontal, symbol Device:R_Small_US
- removed R50: 100, Resistor_THT:R_Axial_DIN0207_L6.3mm_D2.5mm_P7.62mm_Horizontal, symbol Device:R_Small_US
- removed R69: 820, Resistor_THT:R_Axial_DIN0207_L6.3mm_D2.5mm_P7.62mm_Horizontal, symbol Device:R_Small_US
- removed R75, R75A1, R75B1, R75C1, R75D1, R75E1, R75F1, R78, R79, R83: 33, Resistor_THT:R_Axial_DIN0207_L6.3mm_D2.5mm_P7.62mm_Horizontal, symbol Device:R_Small_US
- removed R8: 18K, Resistor_THT:R_Axial_DIN0207_L6.3mm_D2.5mm_P7.62mm_Horizontal, symbol Device:R_Small_US
- removed R81: 300K, Resistor_THT:R_Axial_DIN0207_L6.3mm_D2.5mm_P7.62mm_Horizontal, symbol Device:R_Small_US
- removed R82: 82K, Resistor_THT:R_Axial_DIN0207_L6.3mm_D2.5mm_P7.62mm_Horizontal, symbol Device:R_Small_US
- removed R9: 150, Resistor_THT:R_Axial_DIN0207_L6.3mm_D2.5mm_P7.62mm_Horizontal, symbol Device:R_Small_US
- removed S1: SW_Push, Button_Switch_SMD:SW_SPST_PTS645, symbol Switch:SW_Push
- removed S3: Conn_Coaxial, Button_Switch_SMD:SW_SPST_PTS645, symbol Connector:Conn_Coaxial
- removed U1: MC6809E, Package_DIP:DIP-40_W15.24mm, symbol CPU_NXP_6800:MC6809E
- removed U10: MC6883, Package_DIP:DIP-40_W15.24mm, symbol Roni:MC6883
- removed U11: 74LS138, Package_DIP:DIP-20_W7.62mm, symbol 74xx:74LS138
- removed U12: MC1372P, Package_DIP:DIP-16_W7.62mm_Socket, symbol Roni:MC1372P
- removed U14: LM339, Package_DIP:DIP-16_W7.62mm_Socket, symbol Comparator:LM339
- removed U15: LM741, Package_DIP:DIP-8_W7.62mm, symbol Amplifier_Operational:LM741
- removed U16, U29: 74LS02, Package_DIP:DIP-16_W7.62mm, symbol 74xx:74LS02
- removed U2: MC14050B, Package_DIP:DIP-16_W7.62mm, symbol Roni:MC14050B
- removed U28: ROM EXPANSION, Package_DIP:DIP-16_W7.62mm, symbol Roni:MCM68A364
- removed U3: MCM68A364, Package_DIP:DIP-16_W7.62mm, symbol Roni:MCM68A364
- removed U4, U8: 6821, Package_DIP:DIP-40_W15.24mm, symbol Interface:6821
- removed U5: UM1285-8, Package_DIP:DIP-8_W7.62mm, symbol Roni:UM1285-8
- removed U6: 74LS273, Package_DIP:DIP-20_W7.62mm, symbol 74xx:74LS273
- removed U7: MC6847, Package_DIP:DIP-40_W15.24mm, symbol Roni:MC6847
- removed U9: MC14529, Package_DIP:DIP-20_W7.62mm, symbol 4xxx:14529
- removed U?: CP400_14050B, symbol Roni:CP400_14050B
- removed x1: 14.31818, Package_DIP:DIP-4_W7.62mm, symbol Device:Crystal_GND2
- added C1: C1, symbol Device:C_Small
- added C35: C35, symbol Device:C_Polarized_Small
- added C36: C36, symbol Device:C_Small
- added CN2: CASSETE, symbol Roni:CP400_DIN5_K7
- added D1: D1, Diode_SMD:D_SOD-123, symbol Diode:1N4148W
- added D11: D11, symbol Device:D_Zener
- added D12: D12, Diode_SMD:D_SOD-123, symbol Diode:1N4148W
- added R20: R20, symbol Device:R_Small
- added R21: R21, symbol Device:R_Small
- added R23: R23, symbol Device:R_Small
- added R24: R24, symbol Device:R_Small
- added R37: R37, symbol Device:R_Small
- added R38: R38, symbol Device:R_Small
- added R39: R39, symbol Device:R_Small
- added R40: R40, symbol Device:R_Small
- added R55: R55, symbol Device:R_Small
- added R56: R56, symbol Device:R_Small
- added R74: R74, symbol Device:R_Small
- added RL1: DIPxx-1Axx-12x, Relay_THT:Relay_StandexMeder_DIP_LowProfile, symbol Relay:DIPxx-1Axx-12x
- L3: value 3.3uH -> 3.3uh
- R73: renamed from R?; value R57 -> R73
- gave numbers to parts that had none: 3
Connections:
- net K1 is gone; now on net CNI14-7: L2.1
- net K2 is gone; now on net CNI14-10: L3.1
- net L2 & FOGOD is gone; now on net FOGOD: C33.1, CN6.2
- net L3 & FOGOE is gone; now on an unnamed net: C34.1, CN5.2
- net /IRQA is gone; now on net /IRQ: CI-14.38 (~{IRQA})
- net /IRQB is gone; now on net /IRQ: CI-14.37 (~{IRQB})
- net /MRD is gone; now on net MRD: CI-21.1, CI-21.19
- net +12V: now also CI-16.3 (V+)
- net +5V: now also CI-10.1 (VBB), CI-10.8 (VDD), CI-21.14 (VCC), CI-22.14 (VCC), CI-3.1 (VBB), CI-3.8 (VDD), CI-4.1 (VBB), CI-4.8 (VDD), CI-5.1 (VBB), CI-5.8 (VDD), CI-6.1 (VBB), CI-6.8 (VDD), CI-7.1 (VBB), CI-7.8 (VDD), CI-8.1 (VBB), CI-8.8 (VDD), CI-9.1 (VBB), CI-9.8 (VDD), R73.1, D1.1 (K), R20.1, R37.1, R56.1, RL1.6; no longer CN?.3 (Pin_3)
- net -12V: now also CI-16.12 (V-)
- net 15: now also CI-8.2 (D)
- net 19: now also CI-10.5 (A0), CI-3.5 (A0), CI-4.5 (A0), CI-5.5 (A0), CI-6.5 (A0), CI-7.5 (A0), CI-8.5 (A0), CI-9.5 (A0)
- net 20: now also CI-10.6 (A1), CI-3.6 (A1), CI-4.6 (A1), CI-5.6 (A1), CI-6.6 (A1), CI-7.6 (A1), CI-8.6 (A1), CI-9.6 (A1)
- net 21: now also CI-10.7 (A2), CI-3.7 (A2), CI-4.7 (A2), CI-5.7 (A2), CI-6.7 (A2), CI-7.7 (A2), CI-8.7 (A2), CI-9.7 (A2)
- net 22: now also CI-10.12 (A3), CI-3.12 (A3), CI-4.12 (A3), CI-5.12 (A3), CI-6.12 (A3), CI-7.12 (A3), CI-8.12 (A3), CI-9.12 (A3)
- net 23: now also CI-10.11 (A4), CI-3.11 (A4), CI-4.11 (A4), CI-5.11 (A4), CI-6.11 (A4), CI-7.11 (A4), CI-8.11 (A4), CI-9.11 (A4)
- net 24: now also CI-10.10 (A5), CI-3.10 (A5), CI-4.10 (A5), CI-5.10 (A5), CI-6.10 (A5), CI-7.10 (A5), CI-8.10 (A5), CI-9.10 (A5)
- net 3: now also CI-15.40 (~{HALT}), R14.1
- net 4: now also CI-15.2 (~{NMI}), R13.1
- net 5: now also CI-14.34 (~{RESET}), CI-17.34 (~{RESET})
- net 6: now also C12.1, CI-15.34 (EIN)
- net 7: now also C13.1, CI-15.35 (QIN)
- net CN13-10: now also CN?.3 (Pin_3)
- net CN3-1: now also R30.2
- net GNDREF: now also C33.2, C34.2, CI-21.1 (~{R}), CI-21.2 (D), CI-21.3 (C), CI-21.7 (GND), CI-22.7 (GND), C1.1, C36.2, CN2.4, D11.2 (A), D12.2 (A), R21.2, R24.1, R40.2, R74.2
- net Q0: now also CI-3.14 (Q)
- net Q1: now also CI-4.14 (Q)
- net Q2: now also CI-5.14 (Q)
- net Q3: now also CI-6.14 (Q)
- net Q4: now also CI-7.14 (Q)
- net Q5: now also CI-8.14 (Q)
- net Q6: now also CI-9.14 (Q)
- net Q7: now also CI-10.14 (Q)
- net RESET: no longer CI-14.34 (~{RESET}), CI-17.34 (~{RESET})
- net VCLK: no longer R?.2
- net /CAS: now also CI-10.15 (/CAS), CI-3.15 (/CAS), CI-4.15 (/CAS), CI-5.15 (/CAS), CI-6.15 (/CAS), CI-7.15 (/CAS), CI-8.15 (/CAS), CI-9.15 (/CAS)
- net /FIRQ: now also CI-15.4 (~{FIRQ}), R11.1
- net /IRQ: now also CI-15.3 (~{IRQ}), R12.1
- net /RAS: now also CI-(3/4/5/6/7/8/9/10).4 (/RAS), CI-10.4 (/RAS), CI-29.12 (/RAS), CI-3.4 (/RAS), CI-4.4 (/RAS), CI-5.4 (/RAS), CI-6.4 (/RAS), CI-7.4 (/RAS), CI-8.4 (/RAS), CI-9.4 (/RAS)
- net at TR?.3 (C): now also D1.2 (A), RL1.13, RL1.2
- net at C4.1, CN6.5: now also CI-15.2 (X0)
- net at C42.1, R22.1, R41.2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: now also CI-15.14 (Y0), CI-16.8 (-), R23.1
- net at CI-17.2 (PA0): now also CI-16.13, R55.1, R56.2
- net /WR: now reaches CI-9.3 (R/W)
- net /WR: now also CI-10.3 (R/W), CI-3.3 (R/W), CI-4.3 (R/W), CI-5.3 (R/W), CI-6.3 (R/W), CI-7.3 (R/W), CI-8.3 (R/W)
- net CN10-A7: now reaches CI-9.9 (VCC)
- net CN10-A7: now also CI-(3/4/5/6/7/8/9/10).9 (A7/+5V), CI-10.9 (VCC), CI-3.9 (VCC), CI-4.9 (VCC), CI-5.9 (VCC), CI-6.9 (VCC), CI-7.9 (VCC), CI-8.9 (VCC), CN10.2 (Pin_2)
- net at C5.1, CN6.4: now also CI-15.3 (X1)
- net FOGOD: now reaches L2.2
- net at CI-16.10 (-): now also R37.2, R38.1
- net at CI-16.11 (+): now also R73.2, R55.2, R74.1
- net at C2.1, CN5.4: now also CI-15.5 (X3)
- net MRD: now reaches CI-28.15 (Y0)
- net at C3.1, CN5.5: now also CI-15.4 (X2)
- net at CI-15.13 (Y1): now also R20.2, R21.1
- new net: C1.2, C35.2, CN2.2, R39.2, R40.1
- new net: D12.1 (K), R38.2, R39.1
- new net: C36.1, CN2.1, R23.2, R24.2
- new net: CN2.3, RL1.1, RL1.14
- new net: CN2.5, RL1.7, RL1.8
- new net: C35.1, D11.1 (K)
- no-connect marks 37 -> 19
Other:
- note added: "DRAM CIS 3 to 10 These are placed here to make it possible to assign the footprints for the 4164 RAMs"
- note removed: "*1 Schematic Refers "Z" as pin 10 Should use pin 9 or 10 ?"
- note removed: "1/2W"
- note removed: "16/32K"
- note removed: "4K"
- note removed: "500 OHM ?"
- note removed: "A15 - A0: the schematic has the pins upside down- does not match any 6809 datasheet."
- note removed: "CN12 Ligado a +5V ?"
- note removed: "GROUNDED CASE"
- note removed: "HIGH"
- note removed: "L2: Where is this end connected ? Because L3 is connected to LSW, could be that L2 is connectd to RSW ?"
- note removed: "LOW"
- note removed: "NOTES 1. ON SOME BOARDS, THE FOLLOWING RESISTORS HAVE BEEN REPLACED WITH FERRITE BEADS: R73, R74, R75 (5 beads). R76, R77, R78, R79 and R83 2. R83 IS USED ONLY ON 32K BOARDS 3. THE FOLLOWING CAPACITORS ARE DELETED FOR 32K: C31, C35, C45, C48, C61, C64, C67 and C70 4. ON A 4K RAM, PIN 13 IS CS 5. ON A 32K RAM, PIN 8 IS Vcc. PIN 1 IS N/C AND PIN 9 IS A7"
- note removed: "R20: Is it 380 Ohm ?"
- note removed: "R34/R35/R36: What's the correct resistance?"
- note removed: "R50: Is it connected to +5V? Schematic is not readable."
- note removed: "SPARE GATES"
- note removed: "U16D: Inputs 11/12 are connected together ?"
- note removed: "U6: The pin names does not match the CoCo schematic Exmaple: 4-5 here is 18-5 in schematics."
- moved on the sheet: CI-16C, CI-16E, CI-21A, CI-21C, CI-22E, CI-27B, CI-27C, CI-3

Commit message: Confirmed connection from D21 to R/W
Connections:
- net RESET is gone; now on net 5: C44.1, D17.2 (A), R36.1
- net 18: now also D21.1 (K)
- net 19: now also CI-17.36 (RS0)
- net 20: now also CI-17.35 (RS1)
- net 36: now also CI-28.7 (Y7), CI-28.9 (Y6)
- net 8: now also CI-17.18 (CB1)
- net CN3-5: no longer CI-19.2 (IN+)
- net at CI-16.2, R56.1, R57.2: now also CI-17.40 (CA1)
Other:
- note removed: "D21: Conecta onde?"

Commit message: Validated ci-19 & ci-24 (UA710CP) againts Rev.3 board
Parts:
- removed CI-21: 74LS244, Package_DIP:DIP-22_W7.62mm, symbol Roni:74LS244
- added CI-(3/4/5/6/7/8/9/10)?: 4164, symbol Roni:CP400_4164
- added CI-2: 74LS244, symbol 74xx:74LS244
- added CI-?: 74LS244, Package_DIP:DIP-22_W7.62mm, symbol Roni:74LS244
- added R33: R33, symbol Device:R_Small
- added R34: R34, symbol Device:R_Small
- added R51: R51, symbol Device:R_Small
- added R52: R52, symbol Device:R_Small
Connections:
- net +5V: now also CI-2.20 (VCC), R34.1, R51.1
- net 10: now also CI-(3/4/5/6/7/8/9/10)?.2 (CI-9_DI6), CI-2.16 (O1a), CI-?.3 (1Y)
- net 11: now also CI-(3/4/5/6/7/8/9/10)?.2 (CI-9_DI6), CI-2.3 (O3b), CI-?.10 (2Y)
- net 12: now also CI-(3/4/5/6/7/8/9/10)?.2 (CI-9_DI6), CI-2.14 (O2a), CI-?.5 (3Y)
- net 13: now also CI-(3/4/5/6/7/8/9/10)?.2 (CI-9_DI6), CI-2.5 (O2b), CI-?.16 (4Y)
- net 14: now also CI-(3/4/5/6/7/8/9/10)?.2 (CI-9_DI6), CI-2.12 (O3a), CI-?.7 (5Y)
- net 15: now also CI-(3/4/5/6/7/8/9/10)?.2 (CI-9_DI6), CI-2.7 (O1b), CI-?.14 (6Y)
- net 16: now also CI-(3/4/5/6/7/8/9/10)?.2 (CI-9_DI6), CI-2.18 (O0a), CI-?.8 (7Y)
- net 17: now also CI-(3/4/5/6/7/8/9/10)?.2 (CI-9_DI6), CI-2.9 (O0b), CI-?.12 (8Y)
- net CN3-5: now also CI-19.3 (IN-)
- net GNDREF: now also CI-2.10 (GND), R33.2, R52.2
- net MRD: now also CI-2.1 (OEa), CI-2.19 (OEb), CI-?.1, CI-?.19
- net /RAS: now also CI-(3/4/5/6/7/8/9/10)?.4 (/RAS)
- net at R?.1, R?.1: now also CI-22.8; no longer CI-22.11
- net at CI-22.13: now also CI-19.7 (OUT); no longer CI-27.4 (~{Q})
- net at CI-22.6, D13.2 (A), R47.1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: now also CI-22.11; no longer CI-22.8
- net at CI-19.2 (IN+): now also R33.1, R34.2
- net at CI-22.4: now also CI-23.7 (OUT); no longer CI-19.7 (OUT)
- net at CI-22.10: now also CI-27.4 (~{Q}); no longer CI-23.7 (OUT)
- net at CI-(3/4/5/6/7/8/9/10).14 (CI-9_DO6), CI-24.2 (DD6), CI-24.32 (INV): now also CI-2.2 (I0a)
- net at CI-(3/4/5/6/7/8/9/10).14 (CI-9_DO6), CI-24.7 (DD4): now also CI-2.8 (I3a)
- net at CI-(3/4/5/6/7/8/9/10).14 (CI-9_DO6), CI-24.5 (DD2): now also CI-2.6 (I2a)
- net at CI-(3/4/5/6/7/8/9/10).14 (CI-9_DO6), CI-24.3 (DD0): now also CI-2.4 (I1a)
- net at CI-(3/4/5/6/7/8/9/10).14 (CI-9_DO6), CI-24.4 (DD1): now also CI-2.17 (I3b)
- net at CI-(3/4/5/6/7/8/9/10).14 (CI-9_DO6), CI-24.6 (DD3): now also CI-2.15 (I2b)
- net at CI-(3/4/5/6/7/8/9/10).14 (CI-9_DO6), CI-24.8 (DD5): now also CI-2.13 (I1b)
- net at CI-(3/4/5/6/7/8/9/10).14 (CI-9_DO6), CI-24.34 (/AS), CI-24.40 (DD7): now also CI-2.11 (I0b)
- net at CI-23.3 (IN-): now also R51.2, R52.1
- new net: CI-(3/4/5/6/7/8/9/10)?.14 (CI-9_DO6), CI-?.11 (MD6)
- new net: CI-(3/4/5/6/7/8/9/10)?.14 (CI-9_DO6), CI-?.13 (MD4)
- new net: CI-(3/4/5/6/7/8/9/10)?.14 (CI-9_DO6), CI-?.15 (MD2)
- new net: CI-(3/4/5/6/7/8/9/10)?.14 (CI-9_DO6), CI-?.17 (MD0)
- new net: CI-(3/4/5/6/7/8/9/10)?.14 (CI-9_DO6), CI-?.2 (MD1)
- new net: CI-(3/4/5/6/7/8/9/10)?.14 (CI-9_DO6), CI-?.4 (MD3)
- new net: CI-(3/4/5/6/7/8/9/10)?.14 (CI-9_DO6), CI-?.6 (MD5)
- new net: CI-(3/4/5/6/7/8/9/10)?.14 (CI-9_DO6), CI-?.9 (MD7)
Other:
- note removed: "/MRD conforme maual do CoCo"
- note removed: "16/64K"
- note removed: "C44: Electrolitico ?"
- moved on the sheet: CI-22C, CI-22D

Commit message: some mroe revisioning done
Parts:
- added D6: D6, Diode_SMD:D_SOD-123, symbol Diode:1N4148W
- R7: renamed from R?; value R50 -> R7
- R9: renamed from R?; value R50 -> R9
- gave numbers to parts that had none: 15
- renumbered CI-(3/4/5/6/7/8/9/10) to CI-(3/4/5/6/7/8/9/10)1, XTAL to XTAL1
Connections:
- net +5V: now also R7.2
- net at CI-17.3 (PA1), CI-20.2 (-): no longer R33.2
- net at C6.1, CN7.2, D7.1 (K)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: now also CN2.1 (Pin_1); no longer CN2.2 (Pin_2)
- net at CI-20.3 (+), R32.1: now also R33.2
- net at CI-1.13 (RFT), R7.1: now also D6.2 (A)
- net at CN7.4: now also CN2.2 (Pin_2); no longer CN2.1 (Pin_1)
- net at CI-1.14 (RFT): now also D6.1 (K)
Other:
- note added: "CH 4"
