File: CP 400 COLOR.kicad_pcb (KiCad board)
At the start: 2 copper layers, 255 x 170 mm, 28 parts, among them J1 Conn_02x20_Odd_Even, J2 DB9_Female, J3 DB9_Female, J4 DB9_Female, J5 DB15_Female_HighDensity_Mount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, J6 Conn_Coaxial, J7 Conn_Coaxial, J8 Conn_02x22_Odd_Even, U1 MC6883, U10 EPM3064ALC44-10, U11 EPM3064ALC44-10, U2 MC6809E, U3 AS6C4008-55PCN, U4 2764, U5 2764, U6 MC1372P, U7 6821, U8 MC6847, U9 6821

Commit message: Progressing with schematic for Prologica 12 Rev.3 for CP 400 Color
Parts:
- removed H1: MountingHole, MountingHole:MountingHole_3.2mm_M3
- removed J1: Conn_02x20_Odd_Even, Connector_IDC:IDC-Header_2x20_P2.54mm_Horizontal
- removed J2, J3, J4: DB9_Female, Connector_Dsub:DSUB-9_Female_Horizontal_P2.77x2.54mm_EdgePinOffset9.40mm
- removed J5: DB15_Female_HighDensity_MountingHoles, Connector_Dsub:DSUB-15_Female_Horizontal_P2.77x2.54mm_EdgePinOffset9.40mm
- removed J6, J7: Conn_Coaxial, Connector_BarrelJack:BarrelJack_CUI_PJ-063AH_Horizontal
- removed J8: Conn_02x22_Odd_Even, Connector_IDC:IDC-Header_2x20_P2.54mm_Vertical
- added C1: 1uf, Capacitor_THT:CP_Radial_D5.0mm_P2.50mm, F.Cu at (-483.4, -56.1)
- added C12: 100, Capacitor_THT:CP_Radial_D5.0mm_P2.50mm, F.Cu at (-355.0, -104.4)
- added C2: 10uf, Capacitor_THT:CP_Radial_D5.0mm_P2.50mm, F.Cu at (-400.2, -62.3)
- added C24: 0.1, Capacitor_THT:CP_Radial_D5.0mm_P2.50mm, F.Cu at (-429.4, -32.3)
- added C25: 0.1, Capacitor_THT:CP_Radial_D5.0mm_P2.50mm, F.Cu at (-393.6, -62.3)
- added C3: 100uf, Capacitor_THT:CP_Radial_D5.0mm_P2.50mm, F.Cu at (-483.4, -49.5)
- added C4: 9.35pf, Capacitor_THT:C_Disc_D3.0mm_W2.0mm_P2.50mm, F.Cu at (-435.1, -25.7)
- added C40: 0.1uf, Capacitor_THT:CP_Radial_D5.0mm_P2.50mm, F.Cu at (-389.4, -70.4)
- added C41: 0.1, Capacitor_THT:CP_Radial_D5.0mm_P2.50mm, F.Cu at (-365.5, -96.3)
- added C42: 0.01, Capacitor_THT:C_Disc_D3.0mm_W2.0mm_P2.50mm, F.Cu at (-383.3, -73.8)
- added C43: 0.1, Capacitor_THT:CP_Radial_D5.0mm_P2.50mm, F.Cu at (-376.3, -84.2)
- added C5: 100uf, Capacitor_THT:CP_Radial_D5.0mm_P2.50mm, F.Cu at (-418.6, -40.4)
- added C52: 20pF, Capacitor_THT:C_Disc_D3.0mm_W2.0mm_P2.50mm, F.Cu at (-387.5, -105.9)
- added C53: 56pF, Capacitor_THT:C_Disc_D3.0mm_W2.0mm_P2.50mm, F.Cu at (-370.2, -82.1)
- added C54: 0.02, Capacitor_THT:C_Disc_D3.0mm_W2.0mm_P2.50mm, F.Cu at (-377.2, -79.1)
- added C55: 0.02, Capacitor_THT:C_Disc_D3.0mm_W2.0mm_P2.50mm, F.Cu at (-429.4, -27.2)
- added C56: 0.02, Capacitor_THT:C_Disc_D3.0mm_W2.0mm_P2.50mm, F.Cu at (-344.4, -110.0)
- added C57: 0.01, Capacitor_THT:C_Disc_D3.0mm_W2.0mm_P2.50mm, F.Cu at (-377.7, -73.8)
- added C58: 0.01, Capacitor_THT:C_Disc_D3.0mm_W2.0mm_P2.50mm, F.Cu at (-383.3, -70.2)
- added C6: 25, Capacitor_THT:C_Disc_D3.0mm_W2.0mm_P2.50mm, F.Cu at (-419.2, -35.3)
- added C61: 39pF, Capacitor_THT:C_Disc_D3.0mm_W2.0mm_P2.50mm, F.Cu at (-409.5, -71.9)
- added C73: 56Pf, Capacitor_THT:C_Disc_D3.0mm_W2.0mm_P2.50mm, F.Cu at (-440.7, -25.7)
- added C75: 56pF, Capacitor_THT:C_Disc_D3.0mm_W2.0mm_P2.50mm, F.Cu at (-366.1, -91.3)
- added C78: 0.02, Capacitor_THT:C_Disc_D3.0mm_W2.0mm_P2.50mm, F.Cu at (-394.2, -57.2)
- added C79: 0.02, Capacitor_THT:C_Disc_D3.0mm_W2.0mm_P2.50mm, F.Cu at (-408.4, -46.1)
- added C80: .02uf, Capacitor_THT:C_Disc_D3.0mm_W2.0mm_P2.50mm, F.Cu at (-370.2, -85.7)
- added C81: .02uf, Capacitor_THT:C_Disc_D3.0mm_W2.0mm_P2.50mm, F.Cu at (-359.4, -97.8)
- added C82: .002uf, Capacitor_THT:C_Disc_D3.0mm_W2.0mm_P2.50mm, F.Cu at (-348.9, -105.9)
- added C85: 220pF, Capacitor_THT:C_Disc_D3.0mm_W2.0mm_P2.50mm, F.Cu at (-412.5, -41.9)
- added CI-10: 4164, Package_DIP:DIP-16_W7.62mm, F.Cu at (141.2, 130.7)
- added CI-21: 74LS244, Package_DIP:DIP-22_W7.62mm, F.Cu at (-494.7, -57.3)
- added CI-3: 4164, Package_DIP:DIP-16_W7.62mm, F.Cu at (110.5, 105.8)
- added CI-4: 4164, Package_DIP:DIP-16_W7.62mm, F.Cu at (120.7, 105.8)
- added CI-5: 4164, Package_DIP:DIP-16_W7.62mm, F.Cu at (130.9, 105.8)
- added CI-6: 4164, Package_DIP:DIP-16_W7.62mm, F.Cu at (141.2, 105.8)
- added CI-7: 4164, Package_DIP:DIP-16_W7.62mm, F.Cu at (110.4, 130.6)
- added CI-8: 4164, Package_DIP:DIP-16_W7.62mm, F.Cu at (120.5, 130.7)
- added CI-9: 4164, Package_DIP:DIP-16_W7.62mm, F.Cu at (130.9, 130.7)
- added CR1: 1N4148, Diode_THT:D_DO-35_SOD27_P7.62mm_Horizontal, F.Cu at (-1.80, 54.2)
- added CR10: IN982, Package_TO_SOT_THT:TO-92, F.Cu at (-400.3, -55.8)
- added CR2: 1N4148, Diode_THT:D_DO-35_SOD27_P7.62mm_Horizontal, F.Cu at (-26.7, 71.8)
- added CR3: 1N4148, Diode_THT:D_DO-35_SOD27_P7.62mm_Horizontal, F.Cu at (-28.0, 78.9)
- added CR4: 1N4148, Diode_THT:D_DO-35_SOD27_P7.62mm_Horizontal, F.Cu at (-38.8, 78.1)
- added CR5: 1N4148, Diode_THT:D_DO-35_SOD27_P7.62mm_Horizontal, F.Cu at (-4.34, 65.2)
- added CR6: 1N4148, Diode_THT:D_DO-35_SOD27_P7.62mm_Horizontal, F.Cu at (-38.8, 74.6)
- added CR7: 1N4148, Diode_THT:D_DO-35_SOD27_P7.62mm_Horizontal, F.Cu at (-26.7, 68.2)
- added CR8: 1N4002, Diode_THT:D_DO-41_SOD81_P10.16mm_Horizontal, F.Cu at (-38.5, 54.6)
- added CR9: IN982, Package_TO_SOT_THT:TO-92, F.Cu at (-411.1, -50.4)
- added Q1: MPS3904, Package_TO_SOT_THT:TO-92, F.Cu at (-16.9, 77.3)
- added Q4: 2N2222, Package_TO_SOT_THT:TO-92, F.Cu at (-11.4, 57.9)
- added R1: 100K, Resistor_THT:R_Axial_DIN0207_L6.3mm_D2.5mm_P7.62mm_Horizontal, F.Cu at (-400.7, -71.6)
- added R10: 10K, Resistor_THT:R_Axial_DIN0207_L6.3mm_D2.5mm_P7.62mm_Horizontal, F.Cu at (-443.8, -49.7)
- added R11: 20K, Resistor_THT:R_Axial_DIN0207_L6.3mm_D2.5mm_P7.62mm_Horizontal, F.Cu at (-398.8, -75.7)
- added R12: 40K, Resistor_THT:R_Axial_DIN0207_L6.3mm_D2.5mm_P7.62mm_Horizontal, F.Cu at (-387.8, -97.8)
- added R13: 80K, Resistor_THT:R_Axial_DIN0207_L6.3mm_D2.5mm_P7.62mm_Horizontal, F.Cu at (-376.7, -109.7)
- added R14: 162K, Resistor_THT:R_Axial_DIN0207_L6.3mm_D2.5mm_P7.62mm_Horizontal, F.Cu at (-433.0, -65.9)
- added R15: 324K, Resistor_THT:R_Axial_DIN0207_L6.3mm_D2.5mm_P7.62mm_Horizontal, F.Cu at (-462.3, -37.2)
- added R16: 3.9K, Resistor_THT:R_Axial_DIN0207_L6.3mm_D2.5mm_P7.62mm_Horizontal, F.Cu at (-409.2, -87.8)
- added R17: 470, Resistor_THT:R_Axial_DIN0207_L6.3mm_D2.5mm_P7.62mm_Horizontal, F.Cu at (-376.8, -89.5)
- added R18: 750, Resistor_THT:R_Axial_DIN0207_L6.3mm_D2.5mm_P7.62mm_Horizontal, F.Cu at (-451.5, -31.7)
- added R19: 12K, Resistor_THT:R_Axial_DIN0207_L6.3mm_D2.5mm_P7.62mm_Horizontal, F.Cu at (-440.7, -37.6)
- added R2: 100K, Resistor_THT:R_Axial_DIN0207_L6.3mm_D2.5mm_P7.62mm_Horizontal, F.Cu at (-377.1, -105.7)
- added R20: 360, Resistor_THT:R_Axial_DIN0207_L6.3mm_D2.5mm_P7.62mm_Horizontal, F.Cu at (-365.9, -109.7)
- added R21: 500, Resistor_THT:R_Axial_DIN0207_L6.3mm_D2.5mm_P7.62mm_Horizontal, F.Cu at (-451.4, -43.9)
- added R22: 10K, Resistor_THT:R_Axial_DIN0207_L6.3mm_D2.5mm_P7.62mm_Horizontal, F.Cu at (-462.3, -29.1)
- added R23: 220, Resistor_THT:R_Axial_DIN0207_L6.3mm_D2.5mm_P7.62mm_Horizontal, F.Cu at (-422.3, -53.8)
- added R23a1: 3.9K, Resistor_THT:R_Axial_DIN0207_L6.3mm_D2.5mm_P7.62mm_Horizontal, F.Cu at (-440.7, -45.7)
- added R24: 1.5K, Resistor_THT:R_Axial_DIN0207_L6.3mm_D2.5mm_P7.62mm_Horizontal, F.Cu at (-462.3, -33.1)
- added R25: 1K, Resistor_THT:R_Axial_DIN0207_L6.3mm_D2.5mm_P7.62mm_Horizontal, F.Cu at (-387.8, -101.9)
- added R26: 1K, Resistor_THT:R_Axial_DIN0207_L6.3mm_D2.5mm_P7.62mm_Horizontal, F.Cu at (-419.1, -45.7)
- added R27: 100 1/2W, Resistor_THT:R_Axial_DIN0207_L6.3mm_D2.5mm_P7.62mm_Horizontal, F.Cu at (-462.2, -43.9)
- added R28: 10K, Resistor_THT:R_Axial_DIN0207_L6.3mm_D2.5mm_P7.62mm_Horizontal, F.Cu at (-451.5, -35.8)
- added R29: 10K, Resistor_THT:R_Axial_DIN0207_L6.3mm_D2.5mm_P7.62mm_Horizontal, F.Cu at (-422.3, -49.7)
- added R3: 4.7K, Resistor_THT:R_Axial_DIN0207_L6.3mm_D2.5mm_P7.62mm_Horizontal, F.Cu at (-388.0, -81.6)
- added R30: 1K, Resistor_THT:R_Axial_DIN0207_L6.3mm_D2.5mm_P7.62mm_Horizontal, F.Cu at (-451.5, -27.7)
- added R31: 4.7K, Resistor_THT:R_Axial_DIN0207_L6.3mm_D2.5mm_P7.62mm_Horizontal, F.Cu at (-398.8, -79.7)
- added R32: 4.7K, Resistor_THT:R_Axial_DIN0207_L6.3mm_D2.5mm_P7.62mm_Horizontal, F.Cu at (-409.5, -75.7)
- added R34: 6.2K, Resistor_THT:R_Axial_DIN0207_L6.3mm_D2.5mm_P7.62mm_Horizontal, F.Cu at (-420.3, -80.0)
- added R35: 6.8K, Resistor_THT:R_Axial_DIN0207_L6.3mm_D2.5mm_P7.62mm_Horizontal, F.Cu at (-377.1, -97.6)
- added R36: 56K, Resistor_THT:R_Axial_DIN0207_L6.3mm_D2.5mm_P7.62mm_Horizontal, F.Cu at (-388.0, -77.6)
- added R37: 56K, Resistor_THT:R_Axial_DIN0207_L6.3mm_D2.5mm_P7.62mm_Horizontal, F.Cu at (-422.3, -65.9)
- added R38: 15K, Resistor_THT:R_Axial_DIN0207_L6.3mm_D2.5mm_P7.62mm_Horizontal, F.Cu at (-473.1, -37.2)
- added R39: 1.5MEG, Resistor_THT:R_Axial_DIN0207_L6.3mm_D2.5mm_P7.62mm_Horizontal, F.Cu at (-398.6, -93.8)
- added R4: 4.7K, Resistor_THT:R_Axial_DIN0207_L6.3mm_D2.5mm_P7.62mm_Horizontal, F.Cu at (-355.1, -109.7)
- added R40: 1K, Resistor_THT:R_Axial_DIN0207_L6.3mm_D2.5mm_P7.62mm_Horizontal, F.Cu at (-387.8, -93.8)
- added R41: 24K, Resistor_THT:R_Axial_DIN0207_L6.3mm_D2.5mm_P7.62mm_Horizontal, F.Cu at (-422.3, -57.8)
- added R42: 75K, Resistor_THT:R_Axial_DIN0207_L6.3mm_D2.5mm_P7.62mm_Horizontal, F.Cu at (-443.8, -53.8)
- added R43: 1.5K, Resistor_THT:R_Axial_DIN0207_L6.3mm_D2.5mm_P7.62mm_Horizontal, F.Cu at (-473.1, -33.1)
- added R44: 4.7K, Resistor_THT:R_Axial_DIN0207_L6.3mm_D2.5mm_P7.62mm_Horizontal, F.Cu at (-398.6, -101.9)
- added R45: 180, Resistor_THT:R_Axial_DIN0207_L6.3mm_D2.5mm_P7.62mm_Horizontal, F.Cu at (-411.5, -63.8)
- added R46: 470, Resistor_THT:R_Axial_DIN0207_L6.3mm_D2.5mm_P7.62mm_Horizontal, F.Cu at (-420.3, -75.9)
- added R47: 1.5K, Resistor_THT:R_Axial_DIN0207_L6.3mm_D2.5mm_P7.62mm_Horizontal, F.Cu at (-411.5, -55.7)
- added R48: 10K, Resistor_THT:R_Axial_DIN0207_L6.3mm_D2.5mm_P7.62mm_Horizontal, F.Cu at (-476.4, -71.0)
- added R49: 10M, Resistor_THT:R_Axial_DIN0207_L6.3mm_D2.5mm_P7.62mm_Horizontal, F.Cu at (-443.8, -65.9)
- added R5: 4.7K, Resistor_THT:R_Axial_DIN0207_L6.3mm_D2.5mm_P7.62mm_Horizontal, F.Cu at (-420.3, -71.9)
- added R50: 100, Resistor_THT:R_Axial_DIN0207_L6.3mm_D2.5mm_P7.62mm_Horizontal, F.Cu at (-398.4, -89.7)
- added R51: 10K, Resistor_THT:R_Axial_DIN0207_L6.3mm_D2.5mm_P7.62mm_Horizontal, F.Cu at (-451.5, -39.8)
- added R52: 10K, Resistor_THT:R_Axial_DIN0207_L6.3mm_D2.5mm_P7.62mm_Horizontal, F.Cu at (-440.7, -29.5)
- added R53: 15K, Resistor_THT:R_Axial_DIN0207_L6.3mm_D2.5mm_P7.62mm_Horizontal, F.Cu at (-366.3, -105.7)
- added R54: 15K, Resistor_THT:R_Axial_DIN0207_L6.3mm_D2.5mm_P7.62mm_Horizontal, F.Cu at (-400.7, -67.6)
- added R55: 10M, Resistor_THT:R_Axial_DIN0207_L6.3mm_D2.5mm_P7.62mm_Horizontal, F.Cu at (-433.0, -53.8)
- added R56: 10M, Resistor_THT:R_Axial_DIN0207_L6.3mm_D2.5mm_P7.62mm_Horizontal, F.Cu at (-411.5, -67.8)
- added R57: 1K, Resistor_THT:R_Axial_DIN0207_L6.3mm_D2.5mm_P7.62mm_Horizontal, F.Cu at (-422.3, -61.9)
- added R6: 4.7K, Resistor_THT:R_Axial_DIN0207_L6.3mm_D2.5mm_P7.62mm_Horizontal, F.Cu at (-440.7, -41.6)
- added R68: 10K, Resistor_THT:R_Axial_DIN0207_L6.3mm_D2.5mm_P7.62mm_Horizontal, F.Cu at (-430.0, -37.6)
- added R69: 820, Resistor_THT:R_Axial_DIN0207_L6.3mm_D2.5mm_P7.62mm_Horizontal, F.Cu at (-398.4, -85.7)
- added R7: 4.7K, Resistor_THT:R_Axial_DIN0207_L6.3mm_D2.5mm_P7.62mm_Horizontal, F.Cu at (-433.0, -49.7)
- added R71: 220, Resistor_THT:R_Axial_DIN0207_L6.3mm_D2.5mm_P7.62mm_Horizontal, F.Cu at (-443.8, -57.8)
- added R72: 100K, Resistor_THT:R_Axial_DIN0207_L6.3mm_D2.5mm_P7.62mm_Horizontal, F.Cu at (-411.5, -59.7)
- added R73: 470, Resistor_THT:R_Axial_DIN0207_L6.3mm_D2.5mm_P7.62mm_Horizontal, F.Cu at (-377.1, -101.6)
- added R74: 470, Resistor_THT:R_Axial_DIN0207_L6.3mm_D2.5mm_P7.62mm_Horizontal, F.Cu at (-387.5, -109.7)
- added R75: 33, Resistor_THT:R_Axial_DIN0207_L6.3mm_D2.5mm_P7.62mm_Horizontal, F.Cu at (-494.8, -27.8)
- added R75A1: 33, Resistor_THT:R_Axial_DIN0207_L6.3mm_D2.5mm_P7.62mm_Horizontal, F.Cu at (-473.1, -29.1)
- added R75B1: 33, Resistor_THT:R_Axial_DIN0207_L6.3mm_D2.5mm_P7.62mm_Horizontal, F.Cu at (-387.6, -89.7)
- added R75C1: 33, Resistor_THT:R_Axial_DIN0207_L6.3mm_D2.5mm_P7.62mm_Horizontal, F.Cu at (-443.8, -61.9)
- added R75D1: 33, Resistor_THT:R_Axial_DIN0207_L6.3mm_D2.5mm_P7.62mm_Horizontal, F.Cu at (-376.8, -93.5)
- added R75E1: 33, Resistor_THT:R_Axial_DIN0207_L6.3mm_D2.5mm_P7.62mm_Horizontal, F.Cu at (-366.3, -101.6)
- added R75F1: 33, Resistor_THT:R_Axial_DIN0207_L6.3mm_D2.5mm_P7.62mm_Horizontal, F.Cu at (-433.0, -57.8)
- added R78: 33, Resistor_THT:R_Axial_DIN0207_L6.3mm_D2.5mm_P7.62mm_Horizontal, F.Cu at (-429.9, -41.6)
- added R79: 33, Resistor_THT:R_Axial_DIN0207_L6.3mm_D2.5mm_P7.62mm_Horizontal, F.Cu at (-387.6, -85.7)
- added R8: 18K, Resistor_THT:R_Axial_DIN0207_L6.3mm_D2.5mm_P7.62mm_Horizontal, F.Cu at (-440.7, -33.5)
- added R80: 470, Resistor_THT:R_Axial_DIN0207_L6.3mm_D2.5mm_P7.62mm_Horizontal, F.Cu at (-433.0, -61.9)
- added R81: 300K, Resistor_THT:R_Axial_DIN0207_L6.3mm_D2.5mm_P7.62mm_Horizontal, F.Cu at (-409.5, -79.7)
- added R82: 82K, Resistor_THT:R_Axial_DIN0207_L6.3mm_D2.5mm_P7.62mm_Horizontal, F.Cu at (-398.6, -97.8)
- added R83: 33, Resistor_THT:R_Axial_DIN0207_L6.3mm_D2.5mm_P7.62mm_Horizontal, F.Cu at (-429.9, -45.7)
- added R9: 150, Resistor_THT:R_Axial_DIN0207_L6.3mm_D2.5mm_P7.62mm_Horizontal, F.Cu at (-409.2, -83.8)
- added S1: SW_Push, Button_Switch_SMD:SW_SPST_PTS645, F.Cu at (-394.6, -107.8)
- added S3: Conn_Coaxial, Button_Switch_SMD:SW_SPST_PTS645, F.Cu at (-416.3, -85.9)
- added U12: MC1372P, Package_DIP:DIP-16_W7.62mm_Socket, F.Cu at (-453.3, -109.6)
- added U14: LM339, Package_DIP:DIP-16_W7.62mm_Socket, F.Cu at (-465.0, -109.6)
- added U15: LM741, Package_DIP:DIP-8_W7.62mm, F.Cu at (-476.3, -82.7)
- added U16: 74LS02, Package_DIP:DIP-16_W7.62mm, F.Cu at (-476.3, -65.7)
- added U28: ROM EXPANSION, Package_DIP:DIP-16_W7.62mm, F.Cu at (-454.6, -87.6)
- added U29: 74LS02, Package_DIP:DIP-16_W7.62mm, F.Cu at (-483.9, -43.8)
- added x1: 14.31818, Package_DIP:DIP-4_W7.62mm, F.Cu at (-473.0, -43.8)
- U1: value MC6883 -> MC6809E
- U10: value EPM3064ALC44-10 -> MC6883; footprint Package_LCC:PLCC-44_THT-Socket -> Package_DIP:DIP-40_W15.24mm
- U11: value EPM3064ALC44-10 -> 74LS138; footprint Package_LCC:PLCC-44_THT-Socket -> Package_DIP:DIP-20_W7.62mm
- U2: value MC6809E -> MC14050B; footprint Package_DIP:DIP-40_W15.24mm -> Package_DIP:DIP-16_W7.62mm
- U3: value AS6C4008-55PCN -> MCM68A364; footprint Package_DIP:DIP-32_W15.24mm -> Package_DIP:DIP-16_W7.62mm
- U4: value 2764 -> 6821; footprint Package_DIP:DIP-28_W15.24mm -> Package_DIP:DIP-40_W15.24mm
- U5: value 2764 -> UM1285-8; footprint Package_DIP:DIP-28_W15.24mm -> Package_DIP:DIP-8_W7.62mm
- U6: value MC1372P -> 74LS273; footprint Package_DIP:DIP-14_W7.62mm -> Package_DIP:DIP-20_W7.62mm
- U7: value 6821 -> MC6847
- U8: value MC6847 -> 6821
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Connections:
- U1 pad 1: /A11 -> 33
- U1 pad 10: unconnected-(U1-Pad10) -> 37
- U1 pad 11: unconnected-(U1-Pad11) -> 31
- U1 pad 12: unconnected-(U1-Pad12) -> 30
- U1 pad 13: unconnected-(U1-Pad13) -> 29
- U1 pad 14: unconnected-(U1-Pad14) -> 28
- U1 pad 15: unconnected-(U1-Pad15) -> 27
- U1 pad 16: /A0 -> 26
- U1 pad 17: /A1 -> 25
- U1 pad 18: /A2 -> 24
- U1 pad 19: /A3 -> 23
- U1 pad 2: /A10 -> 4
- U1 pad 20: GND -> 22
- U1 pad 21: /A4 -> 21
- U1 pad 22: /A5 -> 20
- U1 pad 23: /A6 -> 19
- U1 pad 24: /A7 -> 17
- U1 pad 25: unconnected-(U1-Pad25) -> 16
- U1 pad 26: unconnected-(U1-Pad26) -> 15
- U1 pad 27: unconnected-(U1-Pad27) -> 14
- U1 pad 28: /D0 -> 13
- U1 pad 29: /D1 -> 12
- U1 pad 3: /A9 -> /IRQ
- U1 pad 30: /D2 -> 11
- U1 pad 31: /D3 -> 10
- U1 pad 32: /D4 -> 18
- U1 pad 33: /D5 -> unconnected-(U1-Pad33)
- U1 pad 34: /D6 -> 6
- U1 pad 35: /D7 -> 7
- U1 pad 36: /A15 -> unconnected-(U1-Pad36)
- U1 pad 37: /A14 -> 5
- U1 pad 38: /A13 -> unconnected-(U1-Pad38)
- U1 pad 39: /A12 -> 33
- U1 pad 4: /A8 -> /FIRQ
- U1 pad 40: +5V -> 3
- U1 pad 7: unconnected-(U1-Pad7) -> 9
- U1 pad 8: unconnected-(U1-Pad8) -> 39
- U1 pad 9: unconnected-(U1-Pad9) -> 38
- U10 pad 1: unconnected-(U10-Pad1) -> 30
- U10 pad 10: unconnected-(U10-Pad10) -> Net-(R79-Pad2)
- U10 pad 11: unconnected-(U10-Pad11) -> Net-(R78-Pad2)
- U10 pad 12: unconnected-(U10-Pad12) -> *RAS
- U10 pad 13: unconnected-(U10-Pad13) -> Net-(R73-Pad1)
- U10 pad 14: unconnected-(U10-Pad14) -> Net-(R74-Pad1)
- U10 pad 15: unconnected-(U10-Pad15) -> 18
- U10 pad 16: unconnected-(U10-Pad16) -> 19
- U10 pad 17: unconnected-(U10-Pad17) -> 20
- U10 pad 18: unconnected-(U10-Pad18) -> 21
- U10 pad 19: unconnected-(U10-Pad19) -> 22
- U10 pad 2: unconnected-(U10-Pad2) -> 29
- U10 pad 20: unconnected-(U10-Pad20) -> 33
- U10 pad 21: unconnected-(U10-Pad21) -> 23
- U10 pad 22: unconnected-(U10-Pad22) -> 24
- U10 pad 23: unconnected-(U10-Pad23) -> 25
- U10 pad 24: unconnected-(U10-Pad24) -> 26
- U10 pad 25: unconnected-(U10-Pad25) -> Net-(U10-Pad25)
- U10 pad 26: unconnected-(U10-Pad26) -> Net-(U10-Pad26)
- U10 pad 27: unconnected-(U10-Pad27) -> Net-(U10-Pad27)
- U10 pad 28: unconnected-(U10-Pad28) -> Net-(R75F1-Pad2)
- U10 pad 29: unconnected-(U10-Pad29) -> Net-(R75E1-Pad2)
- U10 pad 3: unconnected-(U10-Pad3) -> 28
- U10 pad 30: unconnected-(U10-Pad30) -> Net-(R75D1-Pad2)
- U10 pad 31: unconnected-(U10-Pad31) -> Net-(R75C1-Pad2)
- U10 pad 32: unconnected-(U10-Pad32) -> Net-(R75B1-Pad2)
- U10 pad 33: unconnected-(U10-Pad33) -> Net-(R75A1-Pad2)
- U10 pad 34: unconnected-(U10-Pad34) -> Net-(JP1-Pad3)
- U10 pad 35: unconnected-(U10-Pad35) -> Net-(R83-Pad2)
- U10 pad 36: unconnected-(U10-Pad36) -> 39
- U10 pad 37: unconnected-(U10-Pad37) -> 38
- U10 pad 38: unconnected-(U10-Pad38) -> 37
- U10 pad 39: unconnected-(U10-Pad39) -> 31
- U10 pad 4: unconnected-(U10-Pad4) -> 27
- U10 pad 40: unconnected-(U10-Pad40) -> 9
- U10 pad 5: unconnected-(U10-Pad5) -> Net-(C4-Pad1)
- U10 pad 6: unconnected-(U10-Pad6) -> Net-(R43-Pad1)
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
Commit message: Doing revision; annotations completed
Parts:
- removed C24, C25, C41, C43: 0.1, Capacitor_THT:CP_Radial_D5.0mm_P2.50mm
- removed C53, C75: 56pF, Capacitor_THT:C_Disc_D3.0mm_W2.0mm_P2.50mm
- removed C54, C55, C56, C78, C79: 0.02, Capacitor_THT:C_Disc_D3.0mm_W2.0mm_P2.50mm
- removed C57, C58: 0.01, Capacitor_THT:C_Disc_D3.0mm_W2.0mm_P2.50mm
- removed C61: 39pF, Capacitor_THT:C_Disc_D3.0mm_W2.0mm_P2.50mm
- removed C73: 56Pf, Capacitor_THT:C_Disc_D3.0mm_W2.0mm_P2.50mm
- removed C80, C81: .02uf, Capacitor_THT:C_Disc_D3.0mm_W2.0mm_P2.50mm
- removed C82: .002uf, Capacitor_THT:C_Disc_D3.0mm_W2.0mm_P2.50mm
- removed C85: 220pF, Capacitor_THT:C_Disc_D3.0mm_W2.0mm_P2.50mm
- removed CR1, CR2, CR3, CR4, CR5, CR6, CR7: 1N4148, Diode_THT:D_DO-35_SOD27_P7.62mm_Horizontal
- removed CR10, CR9: IN982, Package_TO_SOT_THT:TO-92
- removed CR8: 1N4002, Diode_THT:D_DO-41_SOD81_P10.16mm_Horizontal
- removed Q1: MPS3904, Package_TO_SOT_THT:TO-92
- removed Q4: 2N2222, Package_TO_SOT_THT:TO-92
- removed R15: 324K, Resistor_THT:R_Axial_DIN0207_L6.3mm_D2.5mm_P7.62mm_Horizontal
- removed R16, R23a1: 3.9K, Resistor_THT:R_Axial_DIN0207_L6.3mm_D2.5mm_P7.62mm_Horizontal
- removed R17, R80: 470, Resistor_THT:R_Axial_DIN0207_L6.3mm_D2.5mm_P7.62mm_Horizontal
- removed R18: 750, Resistor_THT:R_Axial_DIN0207_L6.3mm_D2.5mm_P7.62mm_Horizontal
- removed R19: 12K, Resistor_THT:R_Axial_DIN0207_L6.3mm_D2.5mm_P7.62mm_Horizontal
- removed R2: 100K, Resistor_THT:R_Axial_DIN0207_L6.3mm_D2.5mm_P7.62mm_Horizontal
- removed R28: 10K, Resistor_THT:R_Axial_DIN0207_L6.3mm_D2.5mm_P7.62mm_Horizontal
- removed R75A1, R75B1, R75C1, R75D1, R75E1, R75F1, R78, R79, R83: 33, Resistor_THT:R_Axial_DIN0207_L6.3mm_D2.5mm_P7.62mm_Horizontal
- removed R81: 300K, Resistor_THT:R_Axial_DIN0207_L6.3mm_D2.5mm_P7.62mm_Horizontal
- removed R82: 82K, Resistor_THT:R_Axial_DIN0207_L6.3mm_D2.5mm_P7.62mm_Horizontal
- removed S1: SW_Push, Button_Switch_SMD:SW_SPST_PTS645
- removed S3: Conn_Coaxial, Button_Switch_SMD:SW_SPST_PTS645
- removed U1: MC6809E, Package_DIP:DIP-40_W15.24mm
- removed U10: MC6883, Package_DIP:DIP-40_W15.24mm
- removed U11: 74LS138, Package_DIP:DIP-20_W7.62mm
- removed U12: MC1372P, Package_DIP:DIP-16_W7.62mm_Socket
- removed U14: LM339, Package_DIP:DIP-16_W7.62mm_Socket
- removed U15: LM741, Package_DIP:DIP-8_W7.62mm
- removed U16, U29: 74LS02, Package_DIP:DIP-16_W7.62mm
- removed U2: MC14050B, Package_DIP:DIP-16_W7.62mm
- removed U28: ROM EXPANSION, Package_DIP:DIP-16_W7.62mm
- removed U3: MCM68A364, Package_DIP:DIP-16_W7.62mm
- removed U4, U8: 6821, Package_DIP:DIP-40_W15.24mm
- removed U5: UM1285-8, Package_DIP:DIP-8_W7.62mm
- removed U6: 74LS273, Package_DIP:DIP-20_W7.62mm
- removed U7: MC6847, Package_DIP:DIP-40_W15.24mm
- removed U9: MC14529, Package_DIP:DIP-20_W7.62mm
- removed x1: 14.31818, Package_DIP:DIP-4_W7.62mm
- added CI-1: 1372, Package_DIP:DIP-14_W7.62mm, F.Cu at (132.3, 66.3)
- added CI-11: 2764, Package_DIP:DIP-28_W15.24mm, F.Cu at (155.8, 143.5)
- added CI-12: 2764, Package_DIP:DIP-28_W15.24mm, F.Cu at (135.7, 143.5)
- added CI-13: MC6809E, Package_DIP:DIP-40_W15.24mm, F.Cu at (185.3, 87.3)
- added CI-14: MC6821, Package_DIP:DIP-40_W15.24mm, F.Cu at (69.9, 161.0)
- added CI-15: 14529, Package_DIP:DIP-16_W7.62mm, F.Cu at (109.1, 127.7)
- added CI-16: LM339, Package_DIP:DIP-14_W7.62mm, F.Cu at (115.7, 193.7)
- added CI-17: MC6821, Package_DIP:DIP-40_W15.24mm, F.Cu at (91.3, 160.9)
- added CI-18: 14050B, Package_DIP:DIP-16_W7.62mm, F.Cu at (79.1, 128.0)
- added CI-19: UA710CP, Package_DIP:DIP-8_W7.62mm, F.Cu at (60.1, 102.0)
- added CI-2: 74LS244, Package_DIP:DIP-20_W7.62mm, F.Cu at (93.5, 66.7)
- added CI-20: LM741, Package_DIP:DIP-8_W7.62mm, F.Cu at (60.0, 133.2)
- added CI-22: 74LS125, Package_DIP:DIP-14_W7.62mm, F.Cu at (76.5, 66.7)
- added CI-23: UA710CP, Package_DIP:DIP-8-N7_W7.62mm, F.Cu at (93.8, 101.0)
- added CI-24: MC6847, Package_DIP:DIP-40_W15.24mm, F.Cu at (107.8, 66.3)
- added CI-27: 74LS123, Package_DIP:DIP-16_W7.62mm, F.Cu at (94.5, 127.9)
- added CI-28: 74LS138, Package_DIP:DIP-16_W7.62mm, F.Cu at (146.4, 190.7)
- added CI-29: MC6883, Package_DIP:DIP-40_W15.24mm, F.Cu at (184.8, 149.0)
- added D1: D1, Diode_SMD:D_SOD-123, F.Cu at (-45.6, 113.2)
- added D12: D12, Diode_SMD:D_SOD-123, F.Cu at (-120.3, 169.0)
- added D13: D13, Diode_SMD:D_SOD-123, F.Cu at (-118.8, 165.6)
- added D14: D14, Diode_SMD:D_SOD-123, F.Cu at (-124.6, 165.6)
- added D15: D15, Diode_SMD:D_SOD-123, F.Cu at (-39.8, 113.2)
- added D16: D16, Diode_SMD:D_SOD-123, F.Cu at (-137.6, 171.4)
- added D17: D17, Diode_SMD:D_SOD-123, F.Cu at (-114.6, 169.0)
- added D18: D18, Diode_SMD:D_SOD-123, F.Cu at (-126.1, 171.4)
- added D19: D19, Diode_SMD:D_SOD-123, F.Cu at (-107.3, 165.6)
- added D20: D20, Diode_SMD:D_SOD-123, F.Cu at (-131.8, 171.4)
- added D21: D21, Diode_SMD:D_SOD-123, F.Cu at (-113.1, 165.6)
- added D6: D6, Diode_SMD:D_SOD-123, F.Cu at (-71.5, 150.4)
- added RL1: DIPxx-1Axx-12x, Relay_THT:Relay_StandexMeder_DIP_LowProfile, F.Cu at (-83.6, 151.8)
- added TR1: TR1, Package_TO_SOT_THT:TO-92, F.Cu at (-132.0, 167.2)
- added TR2: TR1, Package_TO_SOT_THT:TO-92, F.Cu at (-138.5, 167.2)
- CI-21: value 74LS244 -> 74LS74; footprint Package_DIP:DIP-22_W7.62mm -> Package_DIP:DIP-14_W7.62mm
- moved CI-21 593.2 mm to (76.9, 101.3)
- moved CI-4 28.4 mm to (142.6, 87.7)
- moved CI-9 28.4 mm to (152.8, 112.6)
- moved CI-7 28.4 mm to (132.3, 112.5)
- moved CI-3 28.4 mm to (132.4, 87.7)
- moved CI-8 28.4 mm to (142.5, 112.6)
- moved CI-10 28.4 mm to (163.1, 112.6)
- moved CI-5 28.4 mm to (152.8, 87.7)
- moved CI-6 28.4 mm to (163.1, 87.7)
Connections:
- CI-10 pad 1: unconnected-(CI-10-Pad1) -> 9
- CI-10 pad 10: unconnected-(CI-10-Pad10) -> 24
- CI-10 pad 11: unconnected-(CI-10-Pad11) -> 23
- CI-10 pad 12: unconnected-(CI-10-Pad12) -> 22
- CI-10 pad 14: unconnected-(CI-10-Pad14) -> Q7
- CI-10 pad 15: unconnected-(CI-10-Pad15) -> /CAS
- CI-10 pad 3: unconnected-(CI-10-Pad3) -> /WR
- CI-10 pad 4: unconnected-(CI-10-Pad4) -> /RAS
- CI-10 pad 5: unconnected-(CI-10-Pad5) -> 19
- CI-10 pad 6: unconnected-(CI-10-Pad6) -> 20
- CI-10 pad 7: unconnected-(CI-10-Pad7) -> 21
- CI-10 pad 8: unconnected-(CI-10-Pad8) -> 9
- CI-10 pad 9: unconnected-(CI-10-Pad9) -> CN10-A7
- CI-21 pad 1: Net-(CI-21-Pad1) -> 33
- CI-21 pad 10: 11 -> 9
- CI-21 pad 11: unconnected-(CI-21-Pad11) -> //HS
- CI-21 pad 12: 17 -> Net-(CI-21-Pad12)
- CI-21 pad 13: unconnected-(CI-21-Pad13) -> 9
- CI-21 pad 14: 15 -> 9
- CI-21 pad 2: unconnected-(CI-21-Pad2) -> 33
- CI-21 pad 3: 10 -> 33
- CI-21 pad 4: unconnected-(CI-21-Pad4) -> Net-(CI-21-Pad4)
- CI-21 pad 5: 12 -> Net-(CI-21-Pad5)
- CI-21 pad 7: 14 -> 33
- CI-21 pad 8: 16 -> Net-(CI-21-Pad12)
- CI-21 pad 9: unconnected-(CI-21-Pad9) -> Net-(CI-21-Pad9)
- CI-3 pad 1: unconnected-(CI-3-Pad1) -> 9
- CI-3 pad 10: unconnected-(CI-3-Pad10) -> 24
- CI-3 pad 11: unconnected-(CI-3-Pad11) -> 23
- CI-3 pad 12: unconnected-(CI-3-Pad12) -> 22
- CI-3 pad 14: unconnected-(CI-3-Pad14) -> Q0
- CI-3 pad 15: unconnected-(CI-3-Pad15) -> /CAS
- CI-3 pad 3: unconnected-(CI-3-Pad3) -> /WR
- CI-3 pad 4: unconnected-(CI-3-Pad4) -> /RAS
- CI-3 pad 5: unconnected-(CI-3-Pad5) -> 19
- CI-3 pad 6: unconnected-(CI-3-Pad6) -> 20
- CI-3 pad 7: unconnected-(CI-3-Pad7) -> 21
- CI-3 pad 8: unconnected-(CI-3-Pad8) -> 9
- CI-3 pad 9: unconnected-(CI-3-Pad9) -> CN10-A7
- CI-4 pad 1: unconnected-(CI-4-Pad1) -> 9
- CI-4 pad 10: unconnected-(CI-4-Pad10) -> 24
- CI-4 pad 11: unconnected-(CI-4-Pad11) -> 23
- CI-4 pad 12: unconnected-(CI-4-Pad12) -> 22
- CI-4 pad 14: unconnected-(CI-4-Pad14) -> Q1
- CI-4 pad 15: unconnected-(CI-4-Pad15) -> /CAS
- CI-4 pad 3: unconnected-(CI-4-Pad3) -> /WR
- CI-4 pad 4: unconnected-(CI-4-Pad4) -> /RAS
- CI-4 pad 5: unconnected-(CI-4-Pad5) -> 19
- CI-4 pad 6: unconnected-(CI-4-Pad6) -> 20
- CI-4 pad 7: unconnected-(CI-4-Pad7) -> 21
- CI-4 pad 8: unconnected-(CI-4-Pad8) -> 9
- CI-4 pad 9: unconnected-(CI-4-Pad9) -> CN10-A7
- CI-5 pad 1: unconnected-(CI-5-Pad1) -> 9
- CI-5 pad 10: unconnected-(CI-5-Pad10) -> 24
- CI-5 pad 11: unconnected-(CI-5-Pad11) -> 23
- CI-5 pad 12: unconnected-(CI-5-Pad12) -> 22
- CI-5 pad 14: unconnected-(CI-5-Pad14) -> Q2
- CI-5 pad 15: unconnected-(CI-5-Pad15) -> /CAS
- CI-5 pad 3: unconnected-(CI-5-Pad3) -> /WR
- CI-5 pad 4: unconnected-(CI-5-Pad4) -> /RAS
- CI-5 pad 5: unconnected-(CI-5-Pad5) -> 19
- CI-5 pad 6: unconnected-(CI-5-Pad6) -> 20
- CI-5 pad 7: unconnected-(CI-5-Pad7) -> 21
- CI-5 pad 8: unconnected-(CI-5-Pad8) -> 9
- CI-5 pad 9: unconnected-(CI-5-Pad9) -> CN10-A7
- CI-6 pad 1: unconnected-(CI-6-Pad1) -> 9
- CI-6 pad 10: unconnected-(CI-6-Pad10) -> 24
- CI-6 pad 11: unconnected-(CI-6-Pad11) -> 23
- CI-6 pad 12: unconnected-(CI-6-Pad12) -> 22
- CI-6 pad 14: unconnected-(CI-6-Pad14) -> Q3
- CI-6 pad 15: unconnected-(CI-6-Pad15) -> /CAS
- CI-6 pad 3: unconnected-(CI-6-Pad3) -> /WR
- CI-6 pad 4: unconnected-(CI-6-Pad4) -> /RAS
- CI-6 pad 5: unconnected-(CI-6-Pad5) -> 19
- CI-6 pad 6: unconnected-(CI-6-Pad6) -> 20
- CI-6 pad 7: unconnected-(CI-6-Pad7) -> 21
- CI-6 pad 8: unconnected-(CI-6-Pad8) -> 9
- CI-6 pad 9: unconnected-(CI-6-Pad9) -> CN10-A7
- CI-7 pad 1: unconnected-(CI-7-Pad1) -> 9
- CI-7 pad 10: unconnected-(CI-7-Pad10) -> 24
- CI-7 pad 11: unconnected-(CI-7-Pad11) -> 23
- CI-7 pad 12: unconnected-(CI-7-Pad12) -> 22
- CI-7 pad 14: unconnected-(CI-7-Pad14) -> Q4
- CI-7 pad 15: unconnected-(CI-7-Pad15) -> /CAS
- CI-7 pad 3: unconnected-(CI-7-Pad3) -> /WR
- CI-7 pad 4: unconnected-(CI-7-Pad4) -> /RAS
- CI-7 pad 5: unconnected-(CI-7-Pad5) -> 19
- CI-7 pad 6: unconnected-(CI-7-Pad6) -> 20
- CI-7 pad 7: unconnected-(CI-7-Pad7) -> 21
- CI-7 pad 8: unconnected-(CI-7-Pad8) -> 9
- CI-7 pad 9: unconnected-(CI-7-Pad9) -> CN10-A7
- CI-8 pad 1: unconnected-(CI-8-Pad1) -> 9
- CI-8 pad 10: unconnected-(CI-8-Pad10) -> 24
- CI-8 pad 11: unconnected-(CI-8-Pad11) -> 23
- CI-8 pad 12: unconnected-(CI-8-Pad12) -> 22
- CI-8 pad 14: unconnected-(CI-8-Pad14) -> Q5
- CI-8 pad 15: unconnected-(CI-8-Pad15) -> /CAS
- CI-8 pad 2: unconnected-(CI-8-Pad2) -> 15
- CI-8 pad 3: unconnected-(CI-8-Pad3) -> /WR
- CI-8 pad 4: unconnected-(CI-8-Pad4) -> /RAS
- CI-8 pad 5: unconnected-(CI-8-Pad5) -> 19
- CI-8 pad 6: unconnected-(CI-8-Pad6) -> 20
- CI-8 pad 7: unconnected-(CI-8-Pad7) -> 21
- CI-8 pad 8: unconnected-(CI-8-Pad8) -> 9
- CI-8 pad 9: unconnected-(CI-8-Pad9) -> CN10-A7
- CI-9 pad 1: unconnected-(CI-9-Pad1) -> 9
- CI-9 pad 10: unconnected-(CI-9-Pad10) -> 24
- CI-9 pad 11: unconnected-(CI-9-Pad11) -> 23
- CI-9 pad 12: unconnected-(CI-9-Pad12) -> 22
- CI-9 pad 14: unconnected-(CI-9-Pad14) -> Q6
- CI-9 pad 15: unconnected-(CI-9-Pad15) -> /CAS
- CI-9 pad 3: unconnected-(CI-9-Pad3) -> /WR
- CI-9 pad 4: unconnected-(CI-9-Pad4) -> /RAS
- CI-9 pad 5: unconnected-(CI-9-Pad5) -> 19
- CI-9 pad 6: unconnected-(CI-9-Pad6) -> 20
- CI-9 pad 7: unconnected-(CI-9-Pad7) -> 21
- CI-9 pad 8: unconnected-(CI-9-Pad8) -> 9
- CI-9 pad 9: unconnected-(CI-9-Pad9) -> CN10-A7

Commit message: Repositioned all mouting holes for the pcb to match the actual CP 400 mounting holes
Parts:
- added H1: MountingHole, MountingHole:MountingHole_3.2mm_M3, F.Cu at (59.7, 58.5)
- moved R10 720.2 mm to (260.5, 100.4)
- moved R26 720.2 mm to (285.2, 104.5)
- moved R34 720.2 mm to (284.0, 70.2)
- moved R42 720.2 mm to (260.5, 96.4)
- moved R46 720.2 mm to (284.0, 74.2)
- moved R49 720.2 mm to (260.5, 84.2)
- moved R5 720.2 mm to (284.0, 78.3)
- moved R52 720.2 mm to (263.6, 120.7)
- moved R71 720.2 mm to (260.5, 92.3)
- moved R8 720.2 mm to (263.6, 116.6)
- moved C3 720.2 mm to (221.0, 100.6)
- moved C4 720.2 mm to (269.2, 124.5)
- moved C5 720.2 mm to (285.7, 109.8)
- moved C6 720.2 mm to (285.1, 114.8)
- moved R14 720.2 mm to (271.3, 84.2)
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Other:
- outline, holes or cut-outs redrawn

Commit message: Mounting holes are final, looks to be in the precise locations for the CP 400 Color case.
Parts:
- removed H1, H2, H4, H5, H6: MountingHole, MountingHole:MountingHole_3.2mm_M3
- removed H3, H7, H8: MountingHole, MountingHole:MountingHole_6.5mm
Other:
- outline, holes or cut-outs redrawn

Commit message: assigned some footprints
Parts:
- added C13: C13, Capacitor_THT:C_Disc_D3.0mm_W1.6mm_P2.50mm, F.Cu at (-62.7, 88.6)
- added C14: C14, Capacitor_THT:C_Disc_D3.0mm_W1.6mm_P2.50mm, F.Cu at (-101.8, 99.7)
- added C15: C16, Capacitor_THT:C_Disc_D3.0mm_W1.6mm_P2.50mm, F.Cu at (-75.0, 94.3)
- added C33: C33, Capacitor_THT:C_Disc_D3.0mm_W1.6mm_P2.50mm, F.Cu at (-57.0, 82.9)
- added C34: C34, Capacitor_THT:C_Disc_D3.0mm_W1.6mm_P2.50mm, F.Cu at (-48.2, 73.2)
- added C35: C35, Capacitor_THT:CP_Radial_Tantal_D10.5mm_P5.00mm, F.Cu at (65.0, 67.5)
- added C36: C36, Capacitor_THT:C_Disc_D3.0mm_W1.6mm_P2.50mm, F.Cu at (-62.7, 85.5)
- added C39: C39, Capacitor_THT:C_Disc_D3.0mm_W1.6mm_P2.50mm, F.Cu at (-82.4, 109.3)
- added C44: C44, Capacitor_THT:C_Disc_D3.0mm_W1.6mm_P2.50mm, F.Cu at (-69.3, 94.3)
- added C45: C45, Capacitor_THT:C_Disc_D3.0mm_W1.6mm_P2.50mm, F.Cu at (-62.7, 82.3)
- added C49: C49, Capacitor_THT:C_Disc_D3.0mm_W1.6mm_P2.50mm, F.Cu at (-48.2, 70.0)
- added C7: C7, Capacitor_THT:C_Disc_D3.0mm_W1.6mm_P2.50mm, F.Cu at (-75.0, 97.5)
- added C8: C8, Capacitor_THT:C_Disc_D3.0mm_W1.6mm_P2.50mm, F.Cu at (-57.0, 79.8)
- added C9: C9, Capacitor_THT:C_Disc_D3.0mm_W1.6mm_P2.50mm, F.Cu at (-57.0, 86.0)
- added CH2: CANAL, Connector_PinHeader_2.54mm:PinHeader_1x03_P2.54mm_Horizontal, F.Cu at (230.0, 55.0)
- added CN1: CN9, Connector_PinHeader_2.54mm:PinHeader_1x03_P2.54mm_Vertical, F.Cu at (-105.7, 105.9)
- added CN10: CN10, Connector_PinHeader_2.54mm:PinHeader_1x03_P2.54mm_Vertical, F.Cu at (205.0, 150.0)
- added CN13: CN13, Connector_PinHeader_2.54mm:PinHeader_1x13_P2.54mm_Vertical, F.Cu at (52.5, 170.0)
- added CN14: CN14, Connector_PinHeader_2.54mm:PinHeader_1x13_P2.54mm_Vertical, F.Cu at (55.0, 170.0)
- added CN2: CASSETE, Connector_PinHeader_2.54mm:PinHeader_1x05_P2.54mm_Vertical, F.Cu at (102.6, 57.5)
- added CN3: CN8, Connector_PinHeader_2.54mm:PinHeader_1x03_P2.54mm_Vertical, F.Cu at (-92.3, 100.4)
- added CN4: RS232, Connector_PinHeader_2.54mm:PinHeader_1x04_P2.54mm_Vertical, F.Cu at (59.7, 76.2)
- added CN5: JOYESQ, Connector_PinHeader_2.54mm:PinHeader_1x05_P2.54mm_Vertical, F.Cu at (125.0, 57.5)
- added CN6: JOYDIR, Connector_PinHeader_2.54mm:PinHeader_1x05_P2.54mm_Vertical, F.Cu at (110.0, 57.5)
- added CN7: CP400_CN7, Connector_PinHeader_2.54mm:PinHeader_1x05_P2.54mm_Vertical, F.Cu at (75.0, 57.5)
- added CN8: CN12, Connector_PinHeader_2.54mm:PinHeader_1x03_P2.54mm_Vertical, F.Cu at (-119.1, 105.9)
- added CV-1: CV-1, Capacitor_THT:C_Axial_L5.1mm_D3.1mm_P7.50mm_Horizontal, F.Cu at (177.5, 170.0)
- added D11: D11, Diode_THT:D_DO-34_SOD68_P7.62mm_Horizontal, F.Cu at (237.5, 169.6)
- added D7: D7, Diode_THT:D_DO-34_SOD68_P7.62mm_Horizontal, F.Cu at (237.5, 160.0)
- added L2: 3.3uh, Inductor_THT:L_Axial_L5.3mm_D2.2mm_P7.62mm_Horizontal_Vishay_IM-1, F.Cu at (57.5, 152.5)
- added L3: 3.3uh, Inductor_THT:L_Axial_L5.3mm_D2.2mm_P7.62mm_Horizontal_Vishay_IM-1, F.Cu at (57.5, 156.2)
- added R33: R33, Resistor_THT:R_Axial_DIN0207_L6.3mm_D2.5mm_P7.62mm_Horizontal, F.Cu at (270.6, 157.2)
- added R58: R58, Resistor_THT:R_Axial_DIN0207_L6.3mm_D2.5mm_P7.62mm_Horizontal, F.Cu at (247.5, 177.4)
- added R59: R59, Resistor_THT:R_Axial_DIN0207_L6.3mm_D2.5mm_P7.62mm_Horizontal, F.Cu at (259.8, 157.2)
- added R60: R60, Resistor_THT:R_Axial_DIN0207_L6.3mm_D2.5mm_P7.62mm_Horizontal, F.Cu at (258.2, 177.4)
- added R61: R61, Resistor_THT:R_Axial_DIN0207_L6.3mm_D2.5mm_P7.62mm_Horizontal, F.Cu at (259.8, 165.3)
- added R62: R62, Resistor_THT:R_Axial_DIN0207_L6.3mm_D2.5mm_P7.62mm_Horizontal, F.Cu at (270.6, 161.3)
- added R63: R63, Resistor_THT:R_Axial_DIN0207_L6.3mm_D2.5mm_P7.62mm_Horizontal, F.Cu at (264.9, 169.4)
- added R64: R64, Resistor_THT:R_Axial_DIN0207_L6.3mm_D2.5mm_P7.62mm_Horizontal, F.Cu at (270.6, 165.3)
- added R65: R65, Resistor_THT:R_Axial_DIN0207_L6.3mm_D2.5mm_P7.62mm_Horizontal, F.Cu at (259.8, 161.3)
- added R66: R66, Resistor_THT:R_Axial_DIN0207_L6.3mm_D2.5mm_P7.62mm_Horizontal, F.Cu at (247.5, 181.5)
- added R67: R67, Resistor_THT:R_Axial_DIN0207_L6.3mm_D2.5mm_P7.62mm_Horizontal, F.Cu at (254.2, 173.4)
- added R70: R70, Resistor_THT:R_Axial_DIN0207_L6.3mm_D2.5mm_P7.62mm_Horizontal, F.Cu at (236.7, 176.3)
- added R76: R76, Resistor_THT:R_Axial_DIN0207_L6.3mm_D2.5mm_P7.62mm_Horizontal, F.Cu at (236.7, 180.4)
- added XTAL1: XTAL 1, Crystal:Crystal_AT310_D3.0mm_L10.0mm_Horizontal, F.Cu at (176.2, 175.8)
- C1: value 1uf -> C1; footprint Capacitor_THT:CP_Radial_D5.0mm_P2.50mm -> Capacitor_THT:C_Disc_D3.0mm_W1.6mm_P2.50mm
- C12: value 100 -> C12; footprint Capacitor_THT:CP_Radial_D5.0mm_P2.50mm -> Capacitor_THT:C_Disc_D3.0mm_W1.6mm_P2.50mm
- C2: value 10uf -> C2; footprint Capacitor_THT:CP_Radial_D5.0mm_P2.50mm -> Capacitor_THT:C_Disc_D3.0mm_W1.6mm_P2.50mm
- C3: value 100uf -> C3; footprint Capacitor_THT:CP_Radial_D5.0mm_P2.50mm -> Capacitor_THT:C_Disc_D3.0mm_W1.6mm_P2.50mm
- C4: value 9.35pf -> C4; footprint Capacitor_THT:C_Disc_D3.0mm_W2.0mm_P2.50mm -> Capacitor_THT:C_Disc_D3.0mm_W1.6mm_P2.50mm
- C40: value 0.1uf -> C40; footprint Capacitor_THT:CP_Radial_D5.0mm_P2.50mm -> Capacitor_THT:C_Disc_D3.0mm_W1.6mm_P2.50mm
- C42: value 0.01 -> C42; footprint Capacitor_THT:C_Disc_D3.0mm_W2.0mm_P2.50mm -> Capacitor_THT:C_Disc_D3.0mm_W1.6mm_P2.50mm
- C5: value 100uf -> C5; footprint Capacitor_THT:CP_Radial_D5.0mm_P2.50mm -> Capacitor_THT:C_Disc_D3.0mm_W1.6mm_P2.50mm
- C52: value 20pF -> C52; footprint Capacitor_THT:C_Disc_D3.0mm_W2.0mm_P2.50mm -> Capacitor_THT:C_Disc_D3.0mm_W1.6mm_P2.50mm
- C6: value 25 -> C6; footprint Capacitor_THT:C_Disc_D3.0mm_W2.0mm_P2.50mm -> Capacitor_THT:C_Disc_D3.0mm_W1.6mm_P2.50mm
- D1, D6: footprint Diode_SMD:D_SOD-123 -> Diode_THT:D_DO-34_SOD68_P7.62mm_Horizontal
- D12, D13, D14, D15, D16, D17, D18, D19, D20, D21: footprint Diode_SMD:D_SOD-123 -> Diode_THT:D_DO-34_SOD68_P10.16mm_Horizontal
- R1: value 100K -> R1
- R10: value 10K -> R10
- R11: value 20K -> R11
- R12: value 40K -> R12
- R13: value 80K -> R13
- R14: value 162K -> R14
- R20: value 360 -> R20
- R21: value 500 -> R21
- R22: value 10K -> R22
- R23: value 220 -> R23
- R24: value 1.5K -> R24
- R25: value 1K -> R25
- R26: value 1K -> R26
- R27: value 100 1/2W -> R27
- R29: value 10K -> R29
- R3: value 4.7K -> R3
- R30: value 1K -> R30
- R31: value 4.7K -> R31
- R32: value 4.7K -> R32
- R34: value 6.2K -> R34
- R35: value 6.8K -> R35
- R36: value 56K -> R36
- R37: value 56K -> R37
- R38: value 15K -> R38
- R39: value 1.5MEG -> R39
- R4: value 4.7K -> R4
- R40: value 1K -> R40
- R41: value 24K -> R41
- R42: value 75K -> R42
- R43: value 1.5K -> R43
- R44: value 4.7K -> R44
- R45: value 180 -> R45
- R46: value 470 -> R46
- R47: value 1.5K -> R47
- R48: value 10K -> R48
- R49: value 10M -> R49
- R5: value 4.7K -> R5
- R50: value 100 -> R50
- R51: value 10K -> R51
- R52: value 10K -> R52
- R53: value 15K -> R53
- R54: value 15K -> R54
- R55: value 10M -> R55
- R56: value 10M -> R56
- R57: value 1K -> R57
- R6: value 4.7K -> R6
- R68: value 10K -> R68
- R69: value 820 -> R69
- R7: value 4.7K -> R7
- R71: value 220 -> R71
- R72: value 100K -> R72
- R73: value 470 -> R73
- R74: value 470 -> R74
- R75: value 33 -> R75
- R8: value 18K -> R8
- R9: value 150 -> R9
- moved D19 95.5 mm to (309.9, 60.0)
Connections:
- C1 pad 2: 5 -> Net-(C1-Pad2)
- C12 pad 1: 33 -> 6
- C12 pad 2: Net-(C12-Pad2) -> 33
- C2 pad 2: CSN -> 33
- C3 pad 1: 9 -> Net-(C3-Pad1)
- C40 pad 1: 33 -> Net-(C40-Pad1)
- C40 pad 2: Net-(C40-Pad2) -> 33
- C42 pad 2: Net-(C42-Pad2) -> 33
- C5 pad 1: 9 -> Net-(C5-Pad1)
- C52 pad 1: 33 -> CN3-3
- C52 pad 2: unconnected-(C52-Pad2) -> 33
- C6 pad 1: 33 -> Net-(C6-Pad1)
- C6 pad 2: 9 -> 33
- R1 pad 1: 9 -> 33
- R1 pad 2: Net-(C40-Pad2) -> Net-(CN7-Pad1)
- R10 pad 1: CASSOUT -> 33
- R11 pad 1: CASSOUT -> /FIRQ
- R11 pad 2: Net-(R11-Pad2) -> 9
- R12 pad 1: CASSOUT -> /IRQ
- R12 pad 2: Net-(R12-Pad2) -> 9
- R13 pad 1: CASSOUT -> 4
- R13 pad 2: Net-(R13-Pad2) -> 9
- R14 pad 1: CASSOUT -> 3
- R14 pad 2: Net-(R14-Pad2) -> 9
- R20 pad 1: Net-(CR8-Pad2) -> 9
- R20 pad 2: 9 -> Net-(CI-15-Pad13)
- R21 pad 1: 33 -> Net-(CI-15-Pad13)
- R21 pad 2: Net-(R21-Pad2) -> 33
- R22 pad 1: Net-(R22-Pad1) -> Net-(C42-Pad1)
- R22 pad 2: Net-(R22-Pad2) -> 9
- R23 pad 1: 33 -> Net-(C42-Pad1)
- R23 pad 2: Net-(C2-Pad1) -> Net-(C36-Pad1)
- R24 pad 1: Net-(R23a1-Pad2) -> 33
- R24 pad 2: 33 -> Net-(C36-Pad1)
- R25 pad 1: 9 -> HI
- R25 pad 2: /RS232IN -> 9
- R26 pad 1: 9 -> Net-(CI-17-Pad39)
- R26 pad 2: /CD -> Net-(R26-Pad2)
- R27 pad 1: Net-(P2-Pad4) -> Net-(CI-20-Pad6)
- R29 pad 1: Net-(CR6-Pad1) -> Net-(CI-17-Pad11)
- R29 pad 2: 33 -> Net-(CI-15-Pad10)
- R3 pad 1: 9 -> Net-(C8-Pad1)
- R3 pad 2: 3 -> 2
- R30 pad 1: 9 -> Net-(CI-15-Pad10)
- R30 pad 2: JOYIN -> CN3-1
- R31 pad 1: CSN -> 33
- R31 pad 2: 9 -> CN3-1
- R32 pad 1: 33 -> Net-(CI-20-Pad3)
- R32 pad 2: CSN -> 9
- R34 pad 1: Net-(C2-Pad1) -> Net-(CI-29-Pad6)
- R34 pad 2: Net-(CR4-Pad1) -> Net-(C40-Pad1)
- R35 pad 1: Net-(CR4-Pad1) -> Net-(C45-Pad1)
- R35 pad 2: Net-(R35-Pad2) -> 9
- R36 pad 1: 9 -> 5
- R36 pad 2: Net-(R35-Pad2) -> 9
- R37 pad 2: Net-(R37-Pad2) -> Net-(CI-16-Pad10)
- R38 pad 1: 33 -> Net-(CI-16-Pad10)
- R38 pad 2: Net-(R37-Pad2) -> Net-(D12-Pad1)
- R39 pad 1: CASSDIN -> Net-(D12-Pad1)
- R39 pad 2: Net-(R37-Pad2) -> Net-(C1-Pad2)
- R4 pad 2: 4 -> Net-(C6-Pad1)
- R40 pad 1: 9 -> Net-(C1-Pad2)
- R40 pad 2: CASSDIN -> 33
- R41 pad 1: 33 -> Net-(CI-18-Pad4)
- R41 pad 2: Net-(C82-Pad1) -> Net-(C42-Pad1)
- R42 pad 1: CASSOUT -> Net-(CI-18-Pad10)
- R42 pad 2: Net-(C82-Pad1) -> Net-(C42-Pad1)
- R43 pad 1: Net-(R43-Pad1) -> Net-(CI-18-Pad15)
- R43 pad 2: Net-(C61-Pad2) -> Net-(C42-Pad1)
- R44 pad 1: Net-(R44-Pad1) -> Net-(CI-18-Pad2)
- R44 pad 2: 9 -> Net-(C42-Pad1)
- R45 pad 1: 2 -> Net-(CI-18-Pad6)
- R45 pad 2: Net-(R45-Pad2) -> Net-(C42-Pad1)
- R46 pad 1: Net-(R21-Pad3) -> Net-(CI-18-Pad12)
- R46 pad 2: Net-(Q1-Pad1) -> Net-(C42-Pad1)
- R47 pad 1: 33 -> Net-(CI-22-Pad11)
- R47 pad 2: Net-(Q1-Pad1) -> Net-(CI-1-Pad7)
- R48 pad 1: Net-(R48-Pad1) -> Net-(CI-22-Pad8)
- R48 pad 2: Net-(R48-Pad2) -> Net-(CI-22-Pad11)
- R49 pad 1: Net-(R48-Pad1) -> Net-(CI-22-Pad11)
- R49 pad 2: JOYIN -> Net-(D14-Pad1)
- R5 pad 1: 9 -> Net-(C9-Pad1)
- R5 pad 2: /FIRQ -> unconnected-(R5-Pad2)
- R50 pad 1: 9 -> Net-(CI-22-Pad8)
- R50 pad 2: Net-(C56-Pad2) -> Net-(D13-Pad1)
- R51 pad 1: Net-(R51-Pad1) -> 9
- R51 pad 2: 33 -> Net-(CI-23-Pad3)
- R52 pad 1: Net-(R52-Pad1) -> Net-(CI-23-Pad3)
- R53 pad 1: 9 -> Net-(CI-19-Pad2)
- R53 pad 2: Net-(R51-Pad1) -> 33
- R54 pad 2: Net-(R52-Pad1) -> Net-(CI-19-Pad2)
- R55 pad 1: Net-(R51-Pad1) -> Net-(CI-16-Pad13)
- R55 pad 2: /RS232IN -> Net-(CI-16-Pad11)
- R56 pad 1: Net-(R52-Pad1) -> 9
- R56 pad 2: /CD -> Net-(CI-16-Pad13)
- R57 pad 1: H1 -> Net-(CI-16-Pad5)
- R57 pad 2: 9 -> Net-(CI-16-Pad2)
- R6 pad 1: 9 -> Net-(C15-Pad1)
- R6 pad 2: /IRQ -> Net-(CI-1-Pad10)
- R68 pad 1: 9 -> 33
- R68 pad 2: *CART -> Net-(CI-16-Pad7)
- R69 pad 2: Net-(C12-Pad2) -> Net-(CI-16-Pad5)
- R7 pad 1: 40 -> Net-(CI-1-Pad13)
- R71 pad 1: CASSMOT -> 9
- R71 pad 2: Net-(Q4-Pad2) -> JOYIN
- R72 pad 1: 9 -> Net-(CI-16-Pad9)
- R72 pad 2: CASSOUT -> JOYIN
- R73 pad 1: Net-(R73-Pad1) -> 9
- R73 pad 2: 7 -> Net-(CI-16-Pad11)
- R74 pad 1: Net-(R74-Pad1) -> Net-(CI-16-Pad11)
- R74 pad 2: 6 -> 33
- R75 pad 1: MA6 -> Net-(CI-15-Pad9)
- R75 pad 2: Net-(JP1-Pad2) -> Net-(CI-16-Pad9)
- R8 pad 1: Net-(R21-Pad3) -> Net-(CI-1-Pad12)
- R8 pad 2: Net-(Q1-Pad2) -> Net-(C8-Pad1)
- R9 pad 1: 9 -> Net-(CI-1-Pad12)
- R9 pad 2: Net-(R21-Pad2) -> Net-(R10-Pad2)
