File: CP 400 COLOR.kicad_pcb (KiCad board)
At the start: 2 copper layers, 255 x 170 mm, 154 parts, among them CN1 CN9, CN10 CN10, CN13 CN13, CN14 CN14, CN2 CASSETE, CN3 CN8, CN4 RS232, CN5 JOYESQ, CN6 JOYDIR, CN7 CP400_CN7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

Commit message: Added some components values; Added Photo with component identification in the PCB - WIP
Parts:
- added C8b1: 56pF, Capacitor_THT:C_Disc_D3.0mm_W1.6mm_P2.50mm, F.Cu at (-117.2, 16.4)
- C15: value C16 -> 104
- C39: value C39 -> 220
- C40: value C40 -> 220
- C44: value C44 -> 1Uf 100V; footprint Capacitor_THT:C_Disc_D3.0mm_W1.6mm_P2.50mm -> Capacitor_THT:CP_Axial_L10.0mm_D4.5mm_P15.00mm_Horizontal
- C45: value C45 -> 104
- C7: value C7 -> 100uF; footprint Capacitor_THT:C_Disc_D3.0mm_W1.6mm_P2.50mm -> Capacitor_THT:CP_Radial_Tantal_D10.5mm_P5.00mm
- C8: value C8 -> 104
- C9: value C9 -> 560pF
- CI-18: value 14050B -> CD4050BCN
- CI-23: footprint Package_DIP:DIP-8-N7_W7.62mm -> Package_DIP:DIP-8_W7.62mm
- D15: value D15 -> 1N4148
- D16: value D16 -> 1N4148
- D17: value D17 -> 1N4148
- D6: value D6 -> 1N4002
- D7: value D7 -> 1N4739
- R10: value R10 -> 18K
- R34: value R34 -> 1.5K
- R35: value R35 -> 100K
- R36: value R36 -> 100K
- R5: value R5 -> 470
- R7: value R7 -> 360
- TR1: value TR1 -> F2N3904EBC
- XTAL1: value XTAL 1 -> 14,30244 Mhz
- moved C44 241.6 mm to (156.0, 181.4)
- moved C7 107.5 mm to (-120.4, 0.07)
- moved CI-23 0.53 mm to (59.5, 101.2)
Connections:
- net MRD renamed /MRD
- C45 pad 1: Net-(C45-Pad1) -> CNI13-9
- CI-14 pad 2: CNI14-7 -> CNI14-4
- CI-18 pad 14: Net-(CI-17-Pad4) -> Net-(CI-17-Pad6)
- CI-18 pad 9: Net-(CI-17-Pad6) -> Net-(CI-17-Pad4)
- CI-22 pad 4: Net-(CI-22-Pad4) -> Net-(CI-23-Pad7)
- CN13 pad 1: unconnected-(CN13-Pad1) -> CN13-7
- CN13 pad 9: unconnected-(CN13-Pad9) -> CNI13-9
- CN14 pad 1: unconnected-(CN14-Pad1) -> CN13-3
- CN14 pad 4: unconnected-(CN14-Pad4) -> CNI14-4
- CN14 pad 7: CNI14-7 -> CNI14-4
- CN14 pad 9: unconnected-(CN14-Pad9) -> CN13-8
- D15 pad 1: Net-(C45-Pad1) -> CNI13-9
- D16 pad 2: Net-(C45-Pad1) -> CNI13-9
- D17 pad 1: Net-(C45-Pad1) -> CNI13-9
- L2 pad 1: CNI14-7 -> CNI14-4
- R35 pad 1: Net-(C45-Pad1) -> CNI13-9
- R42 pad 1: Net-(CI-18-Pad10) -> Net-(CI-18-Pad15)
- R43 pad 1: Net-(CI-18-Pad15) -> Net-(CI-18-Pad10)
- R5 pad 2: unconnected-(R5-Pad2) -> /VCLK

Commit message: .
Parts:
- added C10: 104, Capacitor_THT:C_Disc_D3.0mm_W1.6mm_P2.50mm, F.Cu at (-28.6, 50.5)
- C1: value C1 -> 223
- C35: value C35 -> 10uf 25v
- C36: value C36 -> 222
- C49: value C49 -> 152
- D13: value D13 -> 1N4148
- D14: value D14 -> 1N4148
- D20: value D20 -> 1N4148
- D21: value D21 -> 1N4148
- R47, R51, R52, R53, R54: footprint Resistor_THT:R_Axial_DIN0207_L6.3mm_D2.5mm_P7.62mm_Horizontal -> Resistor_THT:R_Axial_DIN0207_L6.3mm_D2.5mm_P5.08mm_Vertical
- R48: value R48 -> 7.5K; footprint Resistor_THT:R_Axial_DIN0207_L6.3mm_D2.5mm_P7.62mm_Horizontal -> Resistor_THT:R_Axial_DIN0207_L6.3mm_D2.5mm_P5.08mm_Vertical
- R49: value R49 -> 4.7K; footprint Resistor_THT:R_Axial_DIN0207_L6.3mm_D2.5mm_P7.62mm_Horizontal -> Resistor_THT:R_Axial_DIN0207_L6.3mm_D2.5mm_P5.08mm_Vertical
- R50: value R50 -> 1.2K; footprint Resistor_THT:R_Axial_DIN0207_L6.3mm_D2.5mm_P7.62mm_Horizontal -> Resistor_THT:R_Axial_DIN0207_L6.3mm_D2.5mm_P5.08mm_Vertical
- R59: value R59 -> 4.7K; footprint Resistor_THT:R_Axial_DIN0207_L6.3mm_D2.5mm_P7.62mm_Horizontal -> Resistor_THT:R_Axial_DIN0207_L6.3mm_D2.5mm_P5.08mm_Vertical
- R60: value R60 -> 3.3K; footprint Resistor_THT:R_Axial_DIN0207_L6.3mm_D2.5mm_P7.62mm_Horizontal -> Resistor_THT:R_Axial_DIN0207_L6.3mm_D2.5mm_P5.08mm_Vertical
- R76: value R76 -> 10K; footprint Resistor_THT:R_Axial_DIN0207_L6.3mm_D2.5mm_P7.62mm_Horizontal -> Resistor_THT:R_Axial_DIN0207_L6.3mm_D2.5mm_P5.08mm_Vertical
- moved C7 78.4 mm to (-55.9, 44.8)
Connections:
- CI-15 pad 13: Net-(CI-15-Pad13) -> Net-(C35-Pad1)
- CI-28 pad 16: unconnected-(CI-28-Pad16) -> 9
- R20 pad 2: Net-(CI-15-Pad13) -> Net-(C35-Pad1)
- R21 pad 1: Net-(CI-15-Pad13) -> Net-(C35-Pad1)
