File: Schematic_No_Video_Mods/CP 400 COLOR.kicad_sch (KiCad schematic)
At the start: 167 parts, among them CN1 CN9, CN10 CN10, CN13 CN13, CN14 CN14, CN2 CASSETE, CN3 CN8, CN4 RS232, CN5 JOYESQ, CN6 JOYDIR, CN8 CN12

Commit message: Add video mods to the schematic
Parts:
- removed Q? (x5): 2N4401, Package_TO_SOT_THT:TO-92_Inline, symbol Transistor_BJT:2N3904
- removed Q?: 2N4403, Package_TO_SOT_THT:TO-92_Inline, symbol Transistor_BJT:2N3905
- removed R?: 4K7, Resistor_THT:R_Axial_DIN0207_L6.3mm_D2.5mm_P7.62mm_Horizontal, symbol Device:R_Small
- removed R?: 150, Resistor_THT:R_Axial_DIN0207_L6.3mm_D2.5mm_P7.62mm_Horizontal, symbol Device:R_Small
- removed R?: 330, Resistor_THT:R_Axial_DIN0207_L6.3mm_D2.5mm_P7.62mm_Horizontal, symbol Device:R_Small
- removed R? (x3): 75, Resistor_THT:R_Axial_DIN0207_L6.3mm_D2.5mm_P7.62mm_Horizontal, symbol Device:R_Small
- removed R? (x3): 1K, Resistor_THT:R_Axial_DIN0207_L6.3mm_D2.5mm_P7.62mm_Horizontal, symbol Device:R_Small
- removed R?: 470, Resistor_THT:R_Axial_DIN0207_L6.3mm_D2.5mm_P7.62mm_Horizontal, symbol Device:R_Small
- removed R?: 10K, Resistor_THT:R_Axial_DIN0207_L6.3mm_D2.5mm_P7.62mm_Horizontal, symbol Device:R_Small
- removed RV?: 1K, symbol Device:R_Potentiometer_US
- removed RV? (x3): 10K, symbol Device:R_Potentiometer_US
- added C16: 56pF, Capacitor_THT:C_Axial_L3.8mm_D2.6mm_P7.50mm_Horizontal, symbol Device:C_Small
- added C8: 104, Capacitor_THT:C_Axial_L3.8mm_D2.6mm_P7.50mm_Horizontal, symbol Device:C_Small
- added CH2: CANAL, Connector_PinHeader_2.54mm:PinHeader_1x03_P2.54mm_Horizontal, symbol Connector:Conn_01x03_Male
- added CN7: CP400_CN7, Connector_PinHeader_2.54mm:PinHeader_1x05_P2.54mm_Vertical, symbol Roni:CP400_CN7
- added D7: 1N4739, Diode_THT:D_DO-34_SOD68_P7.62mm_Horizontal, symbol Device:D_Zener
- added R1: R1, Resistor_THT:R_Axial_DIN0207_L6.3mm_D2.5mm_P7.62mm_Horizontal, symbol Device:R_Small
- added R10: 18K, Resistor_THT:R_Axial_DIN0207_L6.3mm_D2.5mm_P7.62mm_Horizontal, symbol Device:R_Small
- added R3: R3, Resistor_THT:R_Axial_DIN0207_L6.3mm_D2.5mm_P7.62mm_Horizontal, symbol Device:R_Small
- added R8: R8, Resistor_THT:R_Axial_DIN0207_L6.3mm_D2.5mm_P7.62mm_Horizontal, symbol Device:R_Small
- added R9: R9, Resistor_THT:R_Axial_DIN0207_L6.3mm_D2.5mm_P7.62mm_Horizontal, symbol Device:R_Small
- added TR1: F2N3904EBC, Package_TO_SOT_THT:TO-92, symbol Transistor_BJT:MPSA42
- D6: value 1N3064 -> 1N4002
- R6: value 750 -> R6
Connections:
- net +12V: now also R3.2
- net CN3-1: now also CN7.3
- net GNDREF: now also C8.2, CH2.3 (Pin_3), CN7.5, D7.2 (A), R1.1, R10.1
- net at CI-1.12 (RFOut): now also R8.1, R9.1
- net at D14.2 (A), R47.2, R61.1: now also CI-1.7 (0A)
- net at D6.2 (A), R7.1: now also CI-1.13 (RFT); no longer CI-1.14 (RFT)
- net at D6.1 (K): now also CI-1.14 (RFT); no longer CI-1.13 (RFT)
- net CN3-4: now reaches CI-1.5 (0B)
- net CN3-4: now also CI-24.10 (0B)
- net 1372-P9 renamed CN3-6
- new net: C16.2, C8.1, CH2.1 (Pin_1), CN7.2, D7.1 (K), R3.1, R8.2, TR1.3 (C)
- new net: C16.1, R10.2, R9.2, TR1.2 (B)
- new net: CN7.1, R1.2, TR1.1 (E)
- new net: CH2.2 (Pin_2), CN7.4
Other:
- note added: "CH 4"
- note added: "Requer Verificacao"
- note removed: "Composite Video Mod"
- moved on the sheet: D6, R7
